File: pcb/tubes.kicad_sch (KiCad schematic)
At the start: 23 parts, among them Q10 MPSA42, Q11 MPSA42, Q12 MPSA42, Q13 MPSA42, Q4 MPSA42, Q5 MPSA42, Q6 MPSA42, Q7 MPSA42, Q8 MPSA42, Q9 MPSA42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

Commit message: w
Parts:
- added Q14, Q15: MPSA42, Package_TO_SOT_THT:TO-92_Inline, symbol Transistor_BJT:MPSA42
- added R32, R33: 4.7kΩ, Resistor_SMD:R_1206_3216Metric_Pad1.30x1.75mm_HandSolder, symbol Device:R_US
- added U11: CD74HC4067M, Package_SO:SOIC-24W_7.5x15.4mm_P1.27mm, symbol 74xx:CD74HC4067M
- R21: value 33kΩ -> 22kΩ
Connections:
- net NGND: now also Q14.1 (E), Q15.1 (E), U11.12 (GND), U11.15 (~{E})
- net at R22.1: now also U11.22 (I9)
- net at R29.1: now also U11.6 (I3)
- net at R28.1: now also U11.5 (I4)
- net at R23.1: now also U11.9 (I0)
- net at U10.10 (OUTF): now also R33.1
- net at U10.11 (OUTE): now also R32.1
- net at U10.12 (OUTD): now also U11.13 (S3)
- net at U10.13 (OUTC): now also U11.14 (S2)
- net at U10.14 (OUTB): now also U11.11 (S1)
- net at U10.15 (OUTA): now also U11.10 (S0)
- net +5V ISO: now reaches U10.16 (Vcc2)
- net +5V ISO: now also U11.1 (COM), U11.24 (VCC)
- net DIG_A: now reaches U10.2 (INA)
- net DIG_B: now reaches U10.3 (INB)
- net DIG_C: now reaches U10.4 (INC)
- net DIG_D: now reaches U10.5 (IND)
- net LHDP: now reaches U10.6 (INE)
- net RHDP: now reaches U10.7 (INF)
- net at R31.1: now also U11.8 (I1)
- net at R24.1: now also U11.23 (I8)
- net at R25.1: now also U11.2 (I7)
- net at R30.1: now also U11.7 (I2)
- net at N1.LHDP: now also Q14.3 (C)
- net at N1.RHDP: now also Q15.3 (C)
- net at R26.1: now also U11.3 (I6)
- net at R27.1: now also U11.4 (I5)
- new net: Q14.2 (B), R32.2
- new net: Q15.2 (B), R33.2
- no-connect marks 0 -> 6
Other:
- moved on the sheet: R21, U10

Commit message: w
Other:
- moved on the sheet: N1
Changed lines of the file:
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@@
 	(wire
 		(pts
-			(xy 142.24 82.55) (xy 142.24 73.66)
+			(xy 142.24 82.55) (xy 142.24 67.31)
 		)
 		(stroke
@@
 	(wire
 		(pts
+			(xy 336.55 59.69) (xy 336.55 66.04)
+		)
+		(stroke
+			(width 0)
+			(type default)
+		)
+	)
+	(wire
+		(pts
 			(xy 196.85 132.08) (xy 196.85 104.14)
 		)
@@
 	(wire
 		(pts
-			(xy 228.6 82.55) (xy 228.6 63.5)
+			(xy 228.6 82.55) (xy 228.6 57.15)
 		)
 		(stroke
@@
 	(wire
 		(pts
-			(xy 337.82 53.34) (xy 337.82 82.55)
+			(xy 337.82 46.99) (xy 337.82 82.55)
 		)
 		(stroke
@@
 	(wire
 		(pts
-			(xy 359.41 82.55) (xy 359.41 76.2)
+			(xy 359.41 82.55) (xy 359.41 69.85)
 		)
 		(stroke
@@
 	(wire
 		(pts
-			(xy 314.96 53.34) (xy 317.5 53.34)
+			(xy 314.96 46.99) (xy 317.5 46.99)
 		)
 		(stroke
@@
 	(wire
 		(pts
-			(xy 207.01 66.04) (xy 317.5 66.04)
+			(xy 207.01 59.69) (xy 317.5 59.69)
 		)
 		(stroke
@@
 	(wire
 		(pts
+			(xy 336.55 66.04) (xy 369.57 66.04)
+		)
+		(stroke
+			(width 0)
+			(type default)
+		)
+	)
+	(wire
+		(pts
 			(xy 30.48 134.62) (xy 35.56 134.62)
 		)
@@
 	(wire
 		(pts
-			(xy 335.28 66.04) (xy 369.57 66.04)
+			(xy 335.28 59.69) (xy 336.55 59.69)
 		)
 		(stroke
@@
 	(wire
 		(pts
-			(xy 163.83 71.12) (xy 317.5 71.12)
+			(xy 163.83 64.77) (xy 317.5 64.77)
 		)
 		(stroke
@@
 	(wire
 		(pts
-			(xy 185.42 82.55) (xy 185.42 68.58)
+			(xy 185.42 82.55) (xy 185.42 62.23)
 		)
 		(stroke
@@
 	(wire
 		(pts
-			(xy 293.37 82.55) (xy 293.37 55.88)
+			(xy 293.37 82.55) (xy 293.37 49.53)
 		)
 		(stroke
@@
 	(wire
 		(pts
-			(xy 293.37 55.88) (xy 317.5 55.88)
+			(xy 293.37 49.53) (xy 317.5 49.53)
 		)
 		(stroke
@@
 	(wire
 		(pts
-			(xy 359.41 76.2) (xy 335.28 76.2)
+			(xy 359.41 69.85) (xy 335.28 69.85)
 		)
 		(stroke
@@
 	(wire
 		(pts
-			(xy 163.83 82.55) (xy 163.83 71.12)
+			(xy 163.83 82.55) (xy 163.83 64.77)
 		)
 		(stroke
@@
 	(wire
 		(pts
-			(xy 120.65 76.2) (xy 317.5 76.2)
+			(xy 120.65 69.85) (xy 317.5 69.85)
 		)
 		(stroke
@@
 	(wire
 		(pts
-			(xy 142.24 73.66) (xy 317.5 73.66)
+			(xy 142.24 67.31) (xy 317.5 67.31)
 		)
 		(stroke
@@
 	(wire
 		(pts
-			(xy 271.78 58.42) (xy 317.5 58.42)
+			(xy 271.78 52.07) (xy 317.5 52.07)
 		)
 		(stroke
@@
 	(wire
 		(pts
-			(xy 314.96 82.55) (xy 314.96 53.34)
+			(xy 314.96 82.55) (xy 314.96 46.99)
 		)
 		(stroke
@@
 	(wire
 		(pts
-			(xy 207.01 82.55) (xy 207.01 66.04)
+			(xy 207.01 82.55) (xy 207.01 59.69)
 		)
 		(stroke
@@
 	(wire
 		(pts
-			(xy 228.6 63.5) (xy 317.5 63.5)
+			(xy 228.6 57.15) (xy 317.5 57.15)
 		)
 		(stroke
@@
 	(wire
 		(pts
-			(xy 271.78 82.55) (xy 271.78 58.42)
+			(xy 271.78 82.55) (xy 271.78 52.07)
 		)
 		(stroke
@@
 	(wire
 		(pts
-			(xy 250.19 82.55) (xy 250.19 60.96)
+			(xy 250.19 82.55) (xy 250.19 54.61)
 		)
 		(stroke
@@
 	(wire
 		(pts
-			(xy 250.19 60.96) (xy 317.5 60.96)
+			(xy 250.19 54.61) (xy 317.5 54.61)
 		)
 		(stroke
@@
 	(wire
 		(pts
-			(xy 335.28 53.34) (xy 337.82 53.34)
+			(xy 335.28 46.99) (xy 337.82 46.99)
 		)
 		(stroke
@@
 	(wire
 		(pts
-			(xy 120.65 82.55) (xy 120.65 76.2)
+			(xy 120.65 82.55) (xy 120.65 69.85)
 		)
 		(stroke
@@
 	(wire
 		(pts
-			(xy 185.42 68.58) (xy 317.5 68.58)
+			(xy 185.42 62.23) (xy 317.5 62.23)
 		)
 		(stroke
@@
 	(symbol
 		(lib_id "NixiesUS:IN-16")
-		(at 325.12 66.04 0)
+		(at 325.12 59.69 0)
 		(unit 1)
 		(body_style 1)
@@
 		(in_pos_files yes)
 		(dnp no)
-		(fields_autoplaced yes)
 		(property "Reference" "N1"
-			(at 326.39 44.45 0)
+			(at 326.39 36.322 0)
 			(show_name no)
 			(do_not_autoplace no)
@@
 		)
 		(property "Value" "IN-16"
-			(at 325.12 66.04 0)
-			(hide yes)
+			(at 326.39 39.116 0)
 			(show_name no)
 			(do_not_autoplace no)
@@
 					(size 1.143 1.143)
 				)
-				(justify left bottom)
+				(justify bottom)
 			)
 		)
 		(property "Footprint" "nixies-us_IN-16"
-			(at 325.882 62.23 0)
+			(at 325.882 55.88 0)
 			(hide yes)
 			(show_name no)
@@
 		)
 		(property "Datasheet" ""
-			(at 325.12 66.04 0)
+			(at 325.12 59.69 0)
 			(hide yes)
 			(show_name no)
@@
 		)
 		(property "Description" ""
-			(at 325.12 66.04 0)
+			(at 325.12 59.69 0)
 			(hide yes)
 			(show_name no)
@@
 		)
 		(property "Vendor" "Digi-Key"
-			(at 325.12 66.04 0)
+			(at 325.12 59.69 0)
 			(hide yes)
 			(show_name no)

Commit message: fix
Connections:
- net +5V ISO: no longer U11.1 (COM)
- new net PWM: U11.1 (COM)
Changed lines of the file:
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@@
-		(color 0 0 0 0)
-	)
-	(junction
-		(at 88.9 106.68)
-		(diameter 0)
 		(color 0 0 0 0)
 	)
@@
 	(wire
 		(pts
-			(xy 88.9 106.68) (xy 88.9 109.22)
+			(xy 88.9 104.14) (xy 88.9 109.22)
 		)
 		(stroke
@@
 	(wire
 		(pts
-			(xy 88.9 104.14) (xy 88.9 106.68)
-		)
-		(stroke
-			(width 0)
-			(type default)
-		)
-	)
-	(wire
-		(pts
 			(xy 293.37 92.71) (xy 293.37 96.52)
 		)
@@
 	(wire
 		(pts
-			(xy 73.66 121.92) (xy 73.66 106.68)
-		)
-		(stroke
-			(width 0)
-			(type default)
-		)
-	)
-	(wire
-		(pts
 			(xy 185.42 62.23) (xy 317.5 62.23)
 		)
@@
 		(pts
 			(xy 228.6 92.71) (xy 228.6 96.52)
-		)
-		(stroke
-			(width 0)
-			(type default)
-		)
-	)
-	(wire
-		(pts
-			(xy 73.66 106.68) (xy 88.9 106.68)
 		)
 		(stroke
@@
 		(effects
 			(font
+				(size 1.27 1.27)
+			)
+			(justify right)
+		)
+	)
+	(hierarchical_label "PWM"
+		(shape input)
+		(at 73.66 121.92 180)
+		(effects
+			(font
