File: pcb/tubes.kicad_sch (KiCad schematic)
At the start: 28 parts, among them Q10 MPSA42, Q11 MPSA42, Q12 MPSA42, Q13 MPSA42, Q14 MPSA42, Q15 MPSA42, Q4 MPSA42, Q5 MPSA42, Q6 MPSA42, Q7 MPSA42, Q8 MPSA42, Q9 MPSA42, U10 ISO7760DW, U11 CD74HC4067M

Commit message: w
Parts:
- removed Q10, Q11, Q12, Q13, Q14, Q15, Q4, Q5, Q6, Q7, Q8, Q9: MPSA42, Package_TO_SOT_THT:TO-92_Inline, symbol Transistor_BJT:MPSA42
- added Q101, Q107, Q113, Q119, Q125, Q131, Q137, Q143, Q3, Q83, Q89, Q95: MMBTA42, Package_TO_SOT_SMD:SOT-23, symbol Transistor_BJT:MMBTA42
- N1: footprint nixies-us_IN-16 -> nixies-us-IN-16
- R21: footprint Resistor_SMD:R_1206_3216Metric_Pad1.30x1.75mm_HandSolder -> Resistor_SMD:R_2512_6332Metric
- R22, R23, R24, R25, R26, R27, R28, R29, R30, R31, R32, R33: footprint Resistor_SMD:R_1206_3216Metric_Pad1.30x1.75mm_HandSolder -> Resistor_SMD:R_0603_1608Metric
Connections:
- net NGND: now also Q101.2 (E), Q107.2 (E), Q113.2 (E), Q119.2 (E), Q125.2 (E), Q131.2 (E), Q137.2 (E), Q143.2 (E), Q3.2 (E), Q83.2 (E), Q89.2 (E), Q95.2 (E)
- net at R32.2: now also Q137.1 (B)
- net at N1.LHDP: now also Q137.3 (C)
- net at R22.2: now also Q83.1 (B)
- net at R29.2: now also Q119.1 (B)
- net at N1.3: now also Q119.3 (C)
- net at R28.2: now also Q113.1 (B)
- net at N1.4: now also Q113.3 (C)
- net at R23.2: now also Q3.1 (B)
- net at R31.2: now also Q131.1 (B)
- net at R24.2: now also Q89.1 (B)
- net at N1.8: now also Q89.3 (C)
- net at R25.2: now also Q95.1 (B)
- net at R26.2: now also Q101.1 (B)
- net at N1.6: now also Q101.3 (C)
- net at N1.9: now also Q83.3 (C)
- net at R30.2: now also Q125.1 (B)
- net at N1.2: now also Q125.3 (C)
- net at R33.2: now also Q143.1 (B)
- net at N1.RHDP: now also Q143.3 (C)
- net at N1.0: now also Q3.3 (C)
- net at N1.1: now also Q131.3 (C)
- net at N1.5: now also Q107.3 (C)
- net at N1.7: now also Q95.3 (C)
- net at R27.2: now also Q107.1 (B)
Other:
- moved on the sheet: R21
