File: pcb/neon_colon.kicad_sch (KiCad schematic)
At the start: 9 parts, among them Q76 MPSA42, Q77 MPSA42, U22 ISO7760DW

Commit message: w
Parts:
- NE1, NE2: value Lamp_Neon -> NE-2
Changed lines of the file:
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@@
 			)
 		)
-		(property "Value" "Lamp_Neon"
+		(property "Value" "NE-2"
 			(at 191.77 78.7399 0)
 			(show_name no)
@@
 			)
 		)
-		(property "Value" "Lamp_Neon"
+		(property "Value" "NE-2"
 			(at 223.52 97.7899 0)
 			(show_name no)

Commit message: w
Parts:
- R102, R99: value 100kΩ -> 220kΩ
Changed lines of the file:
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@@
 			)
 		)
-		(property "Value" "100kΩ"
+		(property "Value" "220kΩ"
 			(at 222.25 83.8199 0)
 			(show_name no)
@@
 			)
 		)
-		(property "Value" "100kΩ"
+		(property "Value" "220kΩ"
 			(at 190.5 64.7699 0)
 			(show_name no)
