File: pcb/neon_colon.kicad_sch (KiCad schematic)
At the start: 9 parts, among them Q76 MPSA42, Q77 MPSA42, U22 ISO7760DW

Commit message: w
Parts:
- R100, R101, R102, R99: footprint Resistor_SMD:R_1206_3216Metric_Pad1.30x1.75mm_HandSolder -> Resistor_SMD:R_0603_1608Metric
