File: pcb/hv_drive.kicad_sch (KiCad schematic)
At the start: 0 parts

Commit message: w
Parts:
- added C17: 10nF, Capacitor_SMD:C_1206_3216Metric_Pad1.33x1.80mm_HandSolder, symbol Device:C
- added C18: 2200μF, Capacitor_SMD:C_1206_3216Metric_Pad1.33x1.80mm_HandSolder, symbol Device:C_Polarized_US
- added C19, C22, C24, C26: ?F, Capacitor_SMD:C_1206_3216Metric_Pad1.33x1.80mm_HandSolder, symbol Device:C
- added C20: 470μF, Capacitor_SMD:C_1206_3216Metric_Pad1.33x1.80mm_HandSolder, symbol Device:C_Polarized_US
- added C21: 100pF, Capacitor_SMD:C_1206_3216Metric_Pad1.33x1.80mm_HandSolder, symbol Device:C
- added C23: 10μF, Capacitor_SMD:C_1206_3216Metric_Pad1.33x1.80mm_HandSolder, symbol Device:C
- added C25: 6.8μF, Capacitor_SMD:C_1206_3216Metric_Pad1.33x1.80mm_HandSolder, symbol Device:C
- added C27: 1.8nF, Capacitor_SMD:C_1206_3216Metric_Pad1.33x1.80mm_HandSolder, symbol Device:C
- added C28: 330nF, Capacitor_SMD:C_1206_3216Metric_Pad1.33x1.80mm_HandSolder, symbol Device:C
- added C29: 100nF, Capacitor_SMD:C_1206_3216Metric_Pad1.33x1.80mm_HandSolder, symbol Device:C
- added D1: SBR1U400P1, symbol Device:D_Schottky
- added D2: D, symbol Device:D
- added D3: D_Zener, symbol Device:D_Zener
- added D4, D5: 1N5817, Diode_THT:D_DO-41_SOD81_P10.16mm_Horizontal, symbol Diode:1N5817
- added Q1: IGD70R500, Package_TO_SOT_SMD:TO-252-2, symbol Transistor_FET:Q_NMOS_GSD
- added Q2: PNP, symbol Simulation_SPICE:PNP
- added Q3: NPN, symbol Simulation_SPICE:NPN
- added R10, R11, R12, R13, R14, R15, R17, R6, R7, R8, R9: ?Ω, Resistor_SMD:R_1206_3216Metric_Pad1.30x1.75mm_HandSolder, symbol Device:R_US
- added R16: 1.2kΩ, Resistor_SMD:R_1206_3216Metric_Pad1.30x1.75mm_HandSolder, symbol Device:R_US
- added R18: 3.9kΩ, Resistor_SMD:R_1206_3216Metric_Pad1.30x1.75mm_HandSolder, symbol Device:R_US
- added R19: 2.2Ω, Resistor_SMD:R_1206_3216Metric_Pad1.30x1.75mm_HandSolder, symbol Device:R_US
- added R2: 50kΩ, Resistor_SMD:R_1206_3216Metric_Pad1.30x1.75mm_HandSolder, symbol Device:R_US
- added R20: 10Ω, Resistor_SMD:R_1206_3216Metric_Pad1.30x1.75mm_HandSolder, symbol Device:R_US
- added R3: 750mΩ, Resistor_SMD:R_1206_3216Metric_Pad1.30x1.75mm_HandSolder, symbol Device:R_US
- added U5: DA2032-AL, Footprints:DA2032-AL, symbol DA2032-AL:DA2032-AL
- added U6: UA7810, Package_TO_SOT_THT:TO-220-3_Vertical, symbol Regulator_Linear:uA7810
- added U7: TL431DBZ, Package_TO_SOT_SMD:SOT-23, symbol Reference_Voltage:TL431DBZ
- added U8: PC817, Package_DIP:DIP-4_W7.62mm, symbol Isolator:PC817
- added U9: UC3842_SOIC14, Package_SO:SOIC-14_3.9x8.7mm_P1.27mm, symbol Regulator_Controller:UC3842_SOIC14
Connections:
- net VBUS: now also C17.1, C23.1, C28.1, R2.1, U5.10, U5.7, U5.8, U5.9, U6.1 (IN), U9.12 (VCC)
- new net: C24.1, R13.1, R15.1, U9.3 (FB)
- new net: C24.2, Q2.3 (E), R15.2, U9.1 (COMP)
- new net: D1.2 (A), U5.12
- new net: D2.2 (A), Q1.3 (D), U5.3, U5.4, U5.5, U5.6
- new net: C17.2, D2.1 (K), R2.2
- new net: D3.1 (K), R10.1, R7.1, U7.1 (K), U8.2
- new net: C19.2, R6.1, R8.2, U7.2 (REF)
- new net: C25.2, Q2.2 (B), R16.1
- new net: D5.1 (K), R20.1
- new net: C27.1, R18.1, R19.2, R20.2
- new net: D4.2 (A), R19.1
- new net: C26.1, R17.2
- new net: C26.2, Q3.3 (E)
- new net: D4.1 (K), D5.2 (A), U9.10 (OUT)
- new net: C22.2, Q3.2 (B), R12.1, U9.7 (RC)
- new net: Q1.2 (S), R11.2, R3.1
- new net: C21.1, R11.1, R17.1, U9.5 (CS)
- new net: C27.2, Q1.1 (G), R18.2
- new net: C19.1, R7.2
- new net: R13.2, R14.2, U8.3
- new net: R9.2, U8.1
- new net +170V: C18.1, C20.1, D1.1 (K), R10.2, R8.1, R9.1
- new net GND: C21.2, C22.1, C23.2, C25.1, C28.2, C29.2, Q2.1 (C), R14.1, R3.2, U6.2 (GND), U9.8 (PWRGND), U9.9 (GND)
- new net NGND: C18.2, C20.2, D3.2 (A), R6.2, U5.1, U7.3 (A)
- new net VGD: C29.1, U6.3 (OUT), U9.11 (VC)
- new net VREF: Q3.1 (C), R12.2, R16.2, U8.4, U9.14 (VREF)
Other:
- note added: "1:10"

Commit message: w
Parts:
- C22: value ?F -> 1nF
- C26: value ?F -> 10nF
- R11: value ?Ω -> 4.2kΩ
- R12: value ?Ω -> 15.4kΩ
- R17: value ?Ω -> 24.9Ω
Connections:
- net +170V renamed +HVDC
Other:
- added sheet Tubes (tubes.kicad_sch)
- moved on the sheet: C22, C26, Q3, R12, R17

Commit message: w
Parts:
- added C30: 10μF, Capacitor_SMD:C_1206_3216Metric_Pad1.33x1.80mm_HandSolder, symbol Device:C
- added PS1: RSK-2405SRUW_H3, RSK-2405SRUW_H3:CONV_RSK-2405SRUW_H3, symbol RSK-2405SRUW_H3:RSK-2405SRUW_H3
Connections:
- net GND: now also PS1.1 (-VIN)
- net NGND: now also C30.2, PS1.7 (-VOUT)
- net VBUS: now also PS1.2 (+VIN), PS1.3 (CTRL)
- new net: PS1.5 (NC), PS1.8 (NC)
- new net +5V ISO: C30.1, PS1.6 (+VOUT)
Other:
- note added: "180V"

Commit message: work = force * distance
Parts:
- added C31: 10μF, Capacitor_SMD:C_1206_3216Metric_Pad1.33x1.80mm_HandSolder, symbol Device:C
Connections:
- net GND: now also C31.2
- net VBUS: now also C31.1
Other:
- removed sheet Tubes
- moved on the sheet: C17, C18, C19, C20, C21, C22, C23, C24, C25, C26, C27, C30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

Commit message: w
Parts:
- added C32: 10μF, Capacitor_SMD:C_1206_3216Metric_Pad1.33x1.80mm_HandSolder, symbol Device:C
Connections:
- net GND: now also C32.2
- net VGD: now also C32.1
Other:
- moved on the sheet: C17, C23, D2, R2

Commit message: w
Parts:
- removed D2: D, symbol Device:D
- added D7: 1N4148W, Diode_SMD:D_SOD-123, symbol Diode:1N4148W
Connections:
- net at Q1.3 (D), U5.3, U5.4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: now also D7.2 (A)
- net at C17.2, R2.2: now also D7.1 (K)
Changed lines of the file:
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@@
-	)
-	(symbol
-		(lib_id "Device:D")
-		(at 219.71 102.87 270)
-		(unit 1)
-		(body_style 1)
-		(exclude_from_sim no)
-		(in_bom yes)
-		(on_board yes)
-		(in_pos_files yes)
-		(dnp no)
-		(fields_autoplaced yes)
-		(property "Reference" "D2"
-			(at 222.25 101.5999 90)
-			(show_name no)
-			(do_not_autoplace no)
-			(effects
-				(font
-					(size 1.27 1.27)
-				)
-				(justify left)
-			)
-		)
-		(property "Value" "D"
-			(at 222.25 104.1399 90)
-			(show_name no)
-			(do_not_autoplace no)
-			(effects
-				(font
-					(size 1.27 1.27)
-				)
-				(justify left)
-			)
-		)
-		(property "Footprint" ""
-			(at 219.71 102.87 0)
-			(hide yes)
-			(show_name no)
-			(do_not_autoplace no)
-			(effects
-				(font
-					(size 1.27 1.27)
-				)
-			)
-		)
-		(property "Datasheet" ""
-			(at 219.71 102.87 0)
-			(hide yes)
-			(show_name no)
-			(do_not_autoplace no)
-			(effects
-				(font
-					(size 1.27 1.27)
-				)
-			)
-		)
-		(property "Description" "Diode"
-			(at 219.71 102.87 0)
-			(hide yes)
-			(show_name no)
-			(do_not_autoplace no)
-			(effects
-				(font
-					(size 1.27 1.27)
-				)
-			)
-		)
-		(property "Sim.Device" "D"
-			(at 219.71 102.87 0)
-			(hide yes)
-			(show_name no)
-			(do_not_autoplace no)
-			(effects
-				(font
-					(size 1.27 1.27)
-				)
-			)
-		)
-		(property "Sim.Pins" "1=K 2=A"
-			(at 219.71 102.87 0)
-			(hide yes)
-			(show_name no)
-			(do_not_autoplace no)
-			(effects
-				(font
-					(size 1.27 1.27)
-				)
-			)
-		)
-		(pin "2"
-		)
-		(pin "1"
-		)
-		(instances
-			(project "nixie-clock"
-				(path "/ee289ad4-b0b5-4cd2-aa28-bc5cdbd02292/c9568c25-b91e-4e2a-8855-139c3327d912"
-					(reference "D2")
-					(unit 1)
-				)
-			)
-		)
 	)
 	(symbol
@@
 					(unit 1)
 				)
+			)
+		)
+	)
+	(symbol
+		(lib_id "Diode:1N4148W")
+		(at 219.71 102.87 270)
+		(unit 1)
+		(body_style 1)
+		(exclude_from_sim no)
+		(in_bom yes)
+		(on_board yes)
+		(in_pos_files yes)
+		(dnp no)
+		(fields_autoplaced yes)
+		(property "Reference" "D7"
+			(at 222.25 101.5999 90)
+			(show_name no)
+			(do_not_autoplace no)
+			(effects
+				(font
+					(size 1.27 1.27)
+				)
+				(justify left)
+			)
+		)
+		(property "Value" "1N4148W"
+			(at 222.25 104.1399 90)
+			(show_name no)
+			(do_not_autoplace no)
+			(effects
+				(font
+					(size 1.27 1.27)
+				)
+				(justify left)
+			)
+		)
+		(property "Footprint" "Diode_SMD:D_SOD-123"
+			(at 215.265 102.87 0)
+			(hide yes)
+			(show_name no)
+			(do_not_autoplace no)
+			(effects
+				(font
+					(size 1.27 1.27)
+				)
+			)
+		)
+		(property "Datasheet" "https://www.vishay.com/docs/85748/1n4148w.pdf"
+			(at 219.71 102.87 0)
+			(hide yes)
+			(show_name no)
+			(do_not_autoplace no)
+			(effects
+				(font
+					(size 1.27 1.27)
+				)
+			)
+		)
+		(property "Description" "75V 0.15A Fast Switching Diode, SOD-123"
+			(at 219.71 102.87 0)
+			(hide yes)
+			(show_name no)
+			(do_not_autoplace no)
+			(effects
+				(font
+					(size 1.27 1.27)
+				)
+			)
+		)
+		(property "Sim.Device" "D"
+			(at 219.71 102.87 0)
+			(hide yes)
+			(show_name no)
+			(do_not_autoplace no)
+			(effects
+				(font
+					(size 1.27 1.27)
+				)
+			)
+		)
+		(property "Sim.Pins" "1=K 2=A"
+			(at 219.71 102.87 0)
+			(hide yes)
+			(show_name no)
+			(do_not_autoplace no)
+			(effects
+				(font
+					(size 1.27 1.27)
+				)
+			)
+		)
+		(pin "1"
+		)
+		(pin "2"
+		)
+		(instances
+			(project "nixie-clock"
+				(path "/ee289ad4-b0b5-4cd2-aa28-bc5cdbd02292/c9568c25-b91e-4e2a-8855-139c3327d912"
+					(reference "D7")
+					(unit 1)
+				)

Commit message: w
Parts:
- removed C18: 2200μF, Capacitor_SMD:C_1206_3216Metric_Pad1.33x1.80mm_HandSolder, symbol Device:C_Polarized_US
- removed C20: 470μF, Capacitor_SMD:C_1206_3216Metric_Pad1.33x1.80mm_HandSolder, symbol Device:C_Polarized_US
- removed D1: SBR1U400P1, symbol Device:D_Schottky
- removed D3: D_Zener, symbol Device:D_Zener
- removed D4, D5: 1N5817, Diode_THT:D_DO-41_SOD81_P10.16mm_Horizontal, symbol Diode:1N5817
- removed D7: 1N4148W, Diode_SMD:D_SOD-123, symbol Diode:1N4148W
- removed Q1: IGD70R500, Package_TO_SOT_SMD:TO-252-2, symbol Transistor_FET:Q_NMOS_GSD
- removed Q2: PNP, symbol Simulation_SPICE:PNP
- removed Q3: NPN, symbol Simulation_SPICE:NPN
- removed R10, R13, R14, R15, R6, R7, R8, R9: ?Ω, Resistor_SMD:R_1206_3216Metric_Pad1.30x1.75mm_HandSolder, symbol Device:R_US
- removed R11: 4.2kΩ, Resistor_SMD:R_1206_3216Metric_Pad1.30x1.75mm_HandSolder, symbol Device:R_US
- removed R12: 15.4kΩ, Resistor_SMD:R_1206_3216Metric_Pad1.30x1.75mm_HandSolder, symbol Device:R_US
- removed R16: 1.2kΩ, Resistor_SMD:R_1206_3216Metric_Pad1.30x1.75mm_HandSolder, symbol Device:R_US
- removed R17: 24.9Ω, Resistor_SMD:R_1206_3216Metric_Pad1.30x1.75mm_HandSolder, symbol Device:R_US
- removed R18: 3.9kΩ, Resistor_SMD:R_1206_3216Metric_Pad1.30x1.75mm_HandSolder, symbol Device:R_US
- removed R19: 2.2Ω, Resistor_SMD:R_1206_3216Metric_Pad1.30x1.75mm_HandSolder, symbol Device:R_US
- removed R2: 50kΩ, Resistor_SMD:R_1206_3216Metric_Pad1.30x1.75mm_HandSolder, symbol Device:R_US
- removed R20: 10Ω, Resistor_SMD:R_1206_3216Metric_Pad1.30x1.75mm_HandSolder, symbol Device:R_US
- removed R3: 750mΩ, Resistor_SMD:R_1206_3216Metric_Pad1.30x1.75mm_HandSolder, symbol Device:R_US
- removed U6: UA7810, Package_TO_SOT_THT:TO-220-3_Vertical, symbol Regulator_Linear:uA7810
- removed U7: TL431DBZ, Package_TO_SOT_SMD:SOT-23, symbol Reference_Voltage:TL431DBZ
- removed U8: PC817, Package_DIP:DIP-4_W7.62mm, symbol Isolator:PC817
- removed U9: UC3842_SOIC14, Package_SO:SOIC-14_3.9x8.7mm_P1.27mm, symbol Regulator_Controller:UC3842_SOIC14
- added C18: 47nF, Capacitor_SMD:C_1206_3216Metric_Pad1.33x1.80mm_HandSolder, symbol Device:C
- added C20: 680pF, Capacitor_SMD:C_1206_3216Metric_Pad1.33x1.80mm_HandSolder, symbol Device:C
- added C4, C53, C55: 1μF, Capacitor_SMD:C_1206_3216Metric_Pad1.33x1.80mm_HandSolder, symbol Device:C
- added C54, C56: 100nF, Capacitor_SMD:C_1206_3216Metric_Pad1.33x1.80mm_HandSolder, symbol Device:C
- added D1: 1N4150, Diode_SMD:Nexperia_CFP3_SOD-123W, symbol Device:D
- added D2: VS-3EMH06-M3, Diode_SMD:D_SMA_Handsoldering, symbol Device:D
- added Q1: BSC060N10NS3G, Package_TO_SOT_SMD:TDSON-8-1, symbol Transistor_FET:BSC060N10NS3G
- added R119: 33mΩ, Resistor_SMD:R_1206_3216Metric_Pad1.30x1.75mm_HandSolder, symbol Device:R_US
- added R120: 20Ω, Resistor_SMD:R_1206_3216Metric_Pad1.30x1.75mm_HandSolder, symbol Device:R_US
- added R121: 33kΩ, Resistor_SMD:R_1206_3216Metric_Pad1.30x1.75mm_HandSolder, symbol Device:R_US
- added R122: 180kΩ, Resistor_SMD:R_1206_3216Metric_Pad1.30x1.75mm_HandSolder, symbol Device:R_US
- added R123: 5.1kΩ, Resistor_SMD:R_1206_3216Metric_Pad1.30x1.75mm_HandSolder, symbol Device:R_US
- added R124: 1.69MΩ, Resistor_SMD:R_1206_3216Metric_Pad1.30x1.75mm_HandSolder, symbol Device:R_US
- added R125: 10kΩ, Resistor_SMD:R_1206_3216Metric_Pad1.30x1.75mm_HandSolder, symbol Device:R_US
- added U32: LM5156HPWP, Package_SO:Texas_HTSSOP-14-1EP_4.4x5mm_P0.65mm_EP3.4x5mm_Mask3.155x3.255mm_ThermalVias, symbol Regulator_Switching:LM5156HPWP
- added U6: AMC0x11S, symbol Symbols:AMC0x11S
- C17: value 10nF -> 100nF; Manufacturer Part Number (none) -> C1206C104K5RACTU; Vendor Part Number (none) -> 399-C1206C104K5RACTUCT-ND
- C19: value ?F -> 22nF; Manufacturer Part Number (none) -> C1206C104K5RACTU; Vendor Part Number (none) -> 399-C1206C104K5RACTUCT-ND
- C21: value 100pF -> 1μF; Manufacturer Part Number (none) -> CL31B105KAHNNNE; Vendor Part Number (none) -> 1276-1097-1-ND
- C22: value 1nF -> 1μF; Manufacturer Part Number (none) -> CL31B105KAHNNNE; Vendor Part Number (none) -> 1276-1097-1-ND
- C23: Manufacturer Part Number CL31A106MAHNNNE -> CL31B105KAHNNNE; Vendor Part Number 1276-1181-1-ND -> 1276-1097-1-ND
- C24: value ?F -> 10μF; Manufacturer Part Number (none) -> CL31B105KAHNNNE; Vendor Part Number (none) -> 1276-1097-1-ND
- C25: value 6.8μF -> 10μF; Manufacturer Part Number (none) -> CL31B105KAHNNNE; Vendor Part Number (none) -> 1276-1097-1-ND
- C26: value 10nF -> 22nF; Manufacturer Part Number (none) -> C1206C104K5RACTU; Vendor Part Number (none) -> 399-C1206C104K5RACTUCT-ND
- C27: value 1.8nF -> 10nF; Manufacturer Part Number (none) -> C1206C104K5RACTU; Vendor Part Number (none) -> 399-C1206C104K5RACTUCT-ND
- C28: value 330nF -> 220nF; Manufacturer Part Number (none) -> C1206C104K5RACTU; Vendor Part Number (none) -> 399-C1206C104K5RACTUCT-ND
- C29: value 100nF -> 220nF
- C32: value 10μF -> 100pF; Manufacturer Part Number CL31A106MAHNNNE -> (none); Vendor Part Number 1276-1181-1-ND -> (none)
Connections:
- net +5V ISO: now also C53.1, C54.1, U6.1 (VDD1)
- net +HVDC: now also C27.1, C28.1, C29.1, D2.1 (K), R124.2
- net GND: now also C17.2, C19.1, C22.2, C24.2, C25.2, C18.2, C4.2, C55.2, C56.2, R119.2, R121.1, R122.1, U32.15 (AGND), U32.5 (PGND), U32.6 (AGND), U6.3 (REFIN), U6.5 (GND2); no longer C22.1, C25.1, C28.2, C29.2, C32.2
- net NGND: now also C27.2, C28.2, C29.2, C32.1, C53.2, C54.2, R125.1, U6.3 (REFIN), U6.4 (GND1)
- net VBUS: now also C21.1, C22.1, C24.1, C25.1, C26.1, R123.1, U32.1 (BIAS); no longer C28.1
- net at U5.12: now also D2.2 (A)
- net at U5.3, U5.4, U5.5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: now also D1.2 (A), Q1.5 (D)
- net at C19.2: now also R120.1, U32.7 (CS)
- net at C26.2: now also D1.1 (K), R123.2
- removed net VGD: C29.1, C32.1
- new net: C18.1, U32.11 (SS)
- new net: Q1.1 (S), Q1.2 (S), Q1.3 (S), R119.1, R120.2
- new net: C32.2, R124.1, R125.2, U6.2 (OUT)
- new net: C20.2, R121.2
- new net: R122.2, U32.12 (RT)
- new net: C4.1, U32.3 (VCC)
- new net: Q1.4 (G), U32.4 (GATE)
- new net: C20.1, U32.8 (COMP)
- new net +3.3V: C55.1, C56.1, U6.8 (VDD2)
- new net FB: U32.10 (FB), U6.2 (OUT)
Other:
- note added: "170V"
- note added: "Consider BSC059N04LS6ATMA1 BSC067N06LS3GATMA1 BSC060N10NS3GATMA1"
- note removed: "180V"
- moved on the sheet: U5

Commit message: w
Parts:
- added Q2: MMBT3904, Package_TO_SOT_SMD:SOT-23, symbol Transistor_BJT:MMBT3904
- added R126, R127, R128: ?kΩ, Resistor_SMD:R_1206_3216Metric_Pad1.30x1.75mm_HandSolder, symbol Device:R_US
Connections:
- net GND: now also Q2.2 (E), R127.1
- net VBUS: now also R126.2
- net UVLO: now reaches U32.14 (EN/UVLO/SYNC)
- net UVLO: now also Q2.3 (C), R126.1, R127.2
- new net: Q2.1 (B), R128.1
- new net ~{HVDC_EN}: R128.2
Other:
- moved on the sheet: C19
