File: pcb/hv_drive.kicad_sch (KiCad schematic)
At the start: 39 parts, among them Q1 BSC060N10NS3G, Q2 MMBT3904, U32 LM5156HPWP, U5 DA2032-AL, U6 AMC0x11S

Commit message: w
Parts:
- U6: Manufacturer Part Number (none) -> AMC0311S
Changed lines of the file:
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@@
+			)
+		)
+		(property "Manufacturer Part Number" "AMC0311S "
+			(at 246.38 205.74 0)
+			(hide yes)
+			(show_name no)
+			(do_not_autoplace no)
+			(effects
+				(font
+					(size 1.27 1.27)
+				)
 			)
 		)

Commit message: w
Parts:
- C17, C18, C19, C20, C26, C27, C28, C29: Manufacturer Part Number C1206C104K5RACTU -> (none); Vendor Part Number 399-C1206C104K5RACTUCT-ND -> (none)
- C21, C22, C23, C24, C25, C4, C53, C54, C55, C56: Manufacturer Part Number CL31B105KAHNNNE -> (none); Vendor Part Number 1276-1097-1-ND -> (none)
- C30, C31: Manufacturer Part Number CL31A106MAHNNNE -> (none); Vendor Part Number 1276-1181-1-ND -> (none)
- R119, R120, R121, R122, R123, R124, R125, R126, R127, R128: Manufacturer Part Number RMCF1206FT10K0 -> (none); Vendor Part Number RMCF1206FT10K0CT-ND -> (none)
- U6: footprint (none) -> Package_SO:SOIC-8_3.9x4.9mm_P1.27mm
Changed lines of the file:
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@@
 			)
 		)
-		(property "Manufacturer Part Number" "C1206C104K5RACTU"
+		(property "Manufacturer Part Number" ""
 			(at 179.07 151.13 0)
 			(hide yes)
@@
 			)
 		)
-		(property "Vendor Part Number" "399-C1206C104K5RACTUCT-ND"
+		(property "Vendor Part Number" ""
 			(at 179.07 151.13 0)
 			(hide yes)
@@
 			)
 		)
-		(property "Manufacturer Part Number" "CL31A106MAHNNNE"
+		(property "Manufacturer Part Number" ""
 			(at 252.73 48.26 0)
 			(hide yes)
@@
 			)
 		)
-		(property "Vendor Part Number" "1276-1181-1-ND"
+		(property "Vendor Part Number" ""
 			(at 252.73 48.26 0)
 			(hide yes)
@@
 			)
 		)
-		(property "Manufacturer Part Number" "CL31B105KAHNNNE"
+		(property "Manufacturer Part Number" ""
 			(at 132.08 102.87 0)
 			(hide yes)
@@
 			)
 		)
-		(property "Vendor Part Number" "1276-1097-1-ND"
+		(property "Vendor Part Number" ""
 			(at 132.08 102.87 0)
 			(hide yes)
@@
 			)
 		)
-		(property "Manufacturer Part Number" "RMCF1206FT10K0"
+		(property "Manufacturer Part Number" ""
 			(at 213.36 138.43 0)
 			(hide yes)
@@
 			)
 		)
-		(property "Vendor Part Number" "RMCF1206FT10K0CT-ND"
+		(property "Vendor Part Number" ""
 			(at 213.36 138.43 0)
 			(hide yes)
@@
 			)
 		)
-		(property "Manufacturer Part Number" "RMCF1206FT10K0"
+		(property "Manufacturer Part Number" ""
 			(at 222.25 144.78 0)
 			(hide yes)
@@
 			)
 		)
-		(property "Vendor Part Number" "RMCF1206FT10K0CT-ND"
+		(property "Vendor Part Number" ""
 			(at 222.25 144.78 0)
 			(hide yes)
@@
 			)
 		)
-		(property "Manufacturer Part Number" "CL31B105KAHNNNE"
+		(property "Manufacturer Part Number" ""
 			(at 181.61 102.87 0)
 			(hide yes)
@@
 			)
 		)
-		(property "Vendor Part Number" "1276-1097-1-ND"
+		(property "Vendor Part Number" ""
 			(at 181.61 102.87 0)
 			(hide yes)
@@
 			)
 		)
-		(property "Manufacturer Part Number" "RMCF1206FT10K0"
+		(property "Manufacturer Part Number" ""
 			(at 275.59 214.63 0)
 			(hide yes)
@@
 			)
 		)
-		(property "Vendor Part Number" "RMCF1206FT10K0CT-ND"
+		(property "Vendor Part Number" ""
 			(at 275.59 214.63 0)
 			(hide yes)
@@
 			)
 		)
-		(property "Manufacturer Part Number" "RMCF1206FT10K0"
+		(property "Manufacturer Part Number" ""
 			(at 74.93 107.95 0)
 			(hide yes)
@@
 			)
 		)
-		(property "Vendor Part Number" "RMCF1206FT10K0CT-ND"
+		(property "Vendor Part Number" ""
 			(at 74.93 107.95 0)
 			(hide yes)
@@
 			)
 		)
-		(property "Manufacturer Part Number" "C1206C104K5RACTU"
+		(property "Manufacturer Part Number" ""
 			(at 195.58 102.87 0)
 			(hide yes)
@@
 			)
 		)
-		(property "Vendor Part Number" "399-C1206C104K5RACTUCT-ND"
+		(property "Vendor Part Number" ""
 			(at 195.58 102.87 0)
 			(hide yes)
@@
 			)
 		)
-		(property "Manufacturer Part Number" "C1206C104K5RACTU"
+		(property "Manufacturer Part Number" ""
 			(at 205.74 151.13 0)
 			(hide yes)
@@
 			)
 		)
-		(property "Vendor Part Number" "399-C1206C104K5RACTUCT-ND"
+		(property "Vendor Part Number" ""
 			(at 205.74 151.13 0)
 			(hide yes)
@@
 			)
 		)
-		(property "Manufacturer Part Number" "RMCF1206FT10K0"
+		(property "Manufacturer Part Number" ""
 			(at 66.04 139.7 0)
 			(hide yes)
@@
 			)
 		)
-		(property "Vendor Part Number" "RMCF1206FT10K0CT-ND"
+		(property "Vendor Part Number" ""
 			(at 66.04 139.7 0)
 			(hide yes)
@@
 			)
 		)
-		(property "Footprint" ""
+		(property "Footprint" "Package_SO:SOIC-8_3.9x4.9mm_P1.27mm"
 			(at 246.38 205.74 0)
 			(hide yes)
@@
 			)
 		)
-		(property "Manufacturer Part Number" "CL31B105KAHNNNE"
+		(property "Manufacturer Part Number" ""
 			(at 144.78 102.87 0)
 			(hide yes)
@@
 			)
 		)
-		(property "Vendor Part Number" "1276-1097-1-ND"
+		(property "Vendor Part Number" ""
 			(at 144.78 102.87 0)
 			(hide yes)
@@
 			)
 		)
-		(property "Manufacturer Part Number" "C1206C104K5RACTU"
+		(property "Manufacturer Part Number" ""
 			(at 283.21 110.49 0)
 			(hide yes)
@@
 			)
 		)
-		(property "Vendor Part Number" "399-C1206C104K5RACTUCT-ND"
+		(property "Vendor Part Number" ""
 			(at 283.21 110.49 0)
 			(hide yes)
@@
 			)
 		)
-		(property "Manufacturer Part Number" "RMCF1206FT10K0"
+		(property "Manufacturer Part Number" ""
 			(at 193.04 161.29 0)
 			(hide yes)
@@
 			)
 		)
-		(property "Vendor Part Number" "RMCF1206FT10K0CT-ND"
+		(property "Vendor Part Number" ""
 			(at 193.04 161.29 0)
 			(hide yes)
@@
 			)
 		)
-		(property "Manufacturer Part Number" "RMCF1206FT10K0"
+		(property "Manufacturer Part Number" ""
 			(at 275.59 199.39 0)
 			(hide yes)
@@
 			)
 		)
-		(property "Vendor Part Number" "RMCF1206FT10K0CT-ND"
+		(property "Vendor Part Number" ""
 			(at 275.59 199.39 0)
 			(hide yes)
@@
 			)
 		)
-		(property "Manufacturer Part Number" "CL31B105KAHNNNE"
+		(property "Manufacturer Part Number" ""
 			(at 229.87 172.72 0)
 			(hide yes)
@@
 			)
 		)
-		(property "Vendor Part Number" "1276-1097-1-ND"
+		(property "Vendor Part Number" ""
 			(at 229.87 172.72 0)
 			(hide yes)
@@
 			)
 		)
-		(property "Manufacturer Part Number" "C1206C104K5RACTU"
+		(property "Manufacturer Part Number" ""
 			(at 109.22 137.16 0)
 			(hide yes)
@@
 			)
 		)
-		(property "Vendor Part Number" "399-C1206C104K5RACTUCT-ND"
+		(property "Vendor Part Number" ""
 			(at 109.22 137.16 0)
 			(hide yes)
@@
 			)
 		)
-		(property "Manufacturer Part Number" "C1206C104K5RACTU"
+		(property "Manufacturer Part Number" ""
 			(at 308.61 110.49 0)
 			(hide yes)
@@
 			)
 		)
-		(property "Vendor Part Number" "399-C1206C104K5RACTUCT-ND"
+		(property "Vendor Part Number" ""
 			(at 308.61 110.49 0)
 			(hide yes)
@@
 			)
 		)
-		(property "Manufacturer Part Number" "CL31A106MAHNNNE"
+		(property "Manufacturer Part Number" ""
 			(at 200.66 48.26 0)
 			(hide yes)
@@
 			)
 		)
-		(property "Vendor Part Number" "1276-1181-1-ND"
+		(property "Vendor Part Number" ""
 			(at 200.66 48.26 0)
 			(hide yes)
@@
 			)
 		)
-		(property "Manufacturer Part Number" "RMCF1206FT10K0"
+		(property "Manufacturer Part Number" ""
 			(at 74.93 120.65 0)
 			(hide yes)
@@
 			)
 		)
-		(property "Vendor Part Number" "RMCF1206FT10K0CT-ND"
+		(property "Vendor Part Number" ""
 			(at 74.93 120.65 0)
 			(hide yes)
@@
 			)
 		)
-		(property "Manufacturer Part Number" "CL31B105KAHNNNE"
+		(property "Manufacturer Part Number" ""
 			(at 241.3 172.72 0)
 			(hide yes)
@@
 			)
 		)
-		(property "Vendor Part Number" "1276-1097-1-ND"
+		(property "Vendor Part Number" ""
 			(at 241.3 172.72 0)
 			(hide yes)
@@
 			)
 		)
-		(property "Manufacturer Part Number" "RMCF1206FT10K0"
+		(property "Manufacturer Part Number" ""
 			(at 205.74 102.87 0)
 			(hide yes)
@@
 			)
 		)
-		(property "Vendor Part Number" "RMCF1206FT10K0CT-ND"
+		(property "Vendor Part Number" ""
 			(at 205.74 102.87 0)
 			(hide yes)
@@
 			)
 		)
-		(property "Manufacturer Part Number" "CL31B105KAHNNNE"
+		(property "Manufacturer Part Number" ""
 			(at 157.48 102.87 0)
 			(hide yes)
@@
 			)
 		)
-		(property "Vendor Part Number" "1276-1097-1-ND"
+		(property "Vendor Part Number" ""
 			(at 157.48 102.87 0)
 			(hide yes)
@@
 			)
 		)
-		(property "Manufacturer Part Number" "CL31B105KAHNNNE"
+		(property "Manufacturer Part Number" ""
 			(at 251.46 172.72 0)
 			(hide yes)
@@
 			)
 		)
-		(property "Vendor Part Number" "1276-1097-1-ND"
+		(property "Vendor Part Number" ""
 			(at 251.46 172.72 0)
 			(hide yes)
@@
 			)
 		)
-		(property "Manufacturer Part Number" "C1206C104K5RACTU"
+		(property "Manufacturer Part Number" ""
 			(at 295.91 110.49 0)
 			(hide yes)
@@
 			)
 		)
-		(property "Vendor Part Number" "399-C1206C104K5RACTUCT-ND"
+		(property "Vendor Part Number" ""
 			(at 295.91 110.49 0)
 			(hide yes)
@@
 			)
 		)
-		(property "Manufacturer Part Number" "CL31B105KAHNNNE"
+		(property "Manufacturer Part Number" ""
 			(at 170.18 102.87 0)
 			(hide yes)
@@
 			)
 		)
-		(property "Vendor Part Number" "1276-1097-1-ND"
+		(property "Vendor Part Number" ""
 			(at 170.18 102.87 0)
 			(hide yes)
@@
 			)
 		)
-		(property "Manufacturer Part Number" "CL31B105KAHNNNE"
+		(property "Manufacturer Part Number" ""
 			(at 123.19 137.16 0)
 			(hide yes)
@@
 			)
 		)
-		(property "Vendor Part Number" "1276-1097-1-ND"
+		(property "Vendor Part Number" ""
 			(at 123.19 137.16 0)
 			(hide yes)
@@
 			)
 		)
-		(property "Manufacturer Part Number" "C1206C104K5RACTU"
+		(property "Manufacturer Part Number" ""
 			(at 193.04 151.13 0)
 			(hide yes)
@@
 			)
 		)
-		(property "Vendor Part Number" "399-C1206C104K5RACTUCT-ND"
+		(property "Vendor Part Number" ""
 			(at 193.04 151.13 0)
 			(hide yes)
@@
 			)
 		)
-		(property "Manufacturer Part Number" "CL31B105KAHNNNE"
+		(property "Manufacturer Part Number" ""
 			(at 262.89 172.72 0)
 			(hide yes)
@@
 			)
 		)
-		(property "Vendor Part Number" "1276-1097-1-ND"
+		(property "Vendor Part Number" ""
 			(at 262.89 172.72 0)
 			(hide yes)
@@
 			)
 		)
-		(property "Manufacturer Part Number" "RMCF1206FT10K0"
+		(property "Manufacturer Part Number" ""
 			(at 140.97 148.59 0)
 			(hide yes)
@@
 			)
 		)
-		(property "Vendor Part Number" "RMCF1206FT10K0CT-ND"
+		(property "Vendor Part Number" ""
 			(at 140.97 148.59 0)
 			(hide yes)

Commit message: Update hv_drive.kicad_sch
Other:
- note added: "Consider BSC059N04LS6ATMA1 < BSC067N06LS3GATMA1 BSC060N10NS3GATMA1"
- note removed: "Consider BSC059N04LS6ATMA1 BSC067N06LS3GATMA1 BSC060N10NS3GATMA1"
Changed lines of the file:
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@@
 		)
 	)
-	(text "Consider\nBSC059N04LS6ATMA1\nBSC067N06LS3GATMA1\nBSC060N10NS3GATMA1"
+	(text "Consider\nBSC059N04LS6ATMA1 <\nBSC067N06LS3GATMA1\nBSC060N10NS3GATMA1"
 		(exclude_from_sim no)
 		(at 246.888 136.906 0)
