File: pcb/nixie-clock.kicad_sch (KiCad schematic)
At the start: 24 parts, among them J1 USB_C_Receptacle, SW1 SW_Push, U1 TPS25730D, U2 ESP32-S3-WROOM-1, U3 DS3231MZ, U4 STS4X

Commit message: w
Parts:
- SW1: value SW_Push -> Reset
- U3, U4: Vendor (none) -> Digi-Key
Changed lines of the file:
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@@
+			)
+		)
+		(property "Vendor" "Digi-Key"
+			(at 168.91 176.53 0)
+			(hide yes)
+			(show_name no)
+			(do_not_autoplace no)
+			(effects
+				(font
+					(size 1.27 1.27)
+				)
 			)
 		)
@@
 			)
 		)
-		(property "Value" "SW_Push"
+		(property "Value" "Reset"
 			(at 251.46 92.7099 90)
 			(show_name no)
@@
 			(at 217.17 175.26 0)
 			(hide yes)
+			(show_name no)
+			(do_not_autoplace no)
+			(effects
+				(font
+					(size 1.27 1.27)
+				)
+			)
+		)
+		(property "Vendor" "Digi-Key"
+			(at 217.17 175.26 0)
+			(hide yes)

Commit message: w
Parts:
- removed N1: IN-16, nixies-us_IN-16, symbol NixiesUS:IN-16
Changed lines of the file:
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@@
-	)
-	(symbol
-		(lib_id "NixiesUS:IN-16")
-		(at 388.62 120.65 0)
-		(unit 1)
-		(body_style 1)
-		(exclude_from_sim no)
-		(in_bom yes)
-		(on_board yes)
-		(in_pos_files yes)
-		(dnp no)
-		(fields_autoplaced yes)
-		(property "Reference" "N1"
-			(at 389.89 99.06 0)
-			(show_name no)
-			(do_not_autoplace no)
-			(effects
-				(font
-					(size 1.143 1.143)
-				)
-			)
-		)
-		(property "Value" "IN-16"
-			(at 388.62 120.65 0)
-			(hide yes)
-			(show_name no)
-			(do_not_autoplace no)
-			(effects
-				(font
-					(size 1.143 1.143)
-				)
-				(justify left bottom)
-			)
-		)
-		(property "Footprint" "nixies-us_IN-16"
-			(at 389.382 116.84 0)
-			(hide yes)
-			(show_name no)
-			(do_not_autoplace no)
-			(effects
-				(font
-					(size 0.508 0.508)
-				)
-			)
-		)
-		(property "Datasheet" ""
-			(at 388.62 120.65 0)
-			(hide yes)
-			(show_name no)
-			(do_not_autoplace no)
-			(effects
-				(font
-					(size 1.27 1.27)
-				)
-			)
-		)
-		(property "Description" ""
-			(at 388.62 120.65 0)
-			(hide yes)
-			(show_name no)
-			(do_not_autoplace no)
-			(effects
-				(font
-					(size 1.27 1.27)
-				)
-			)
-		)
-		(property "Vendor" "Digi-Key"
-			(at 388.62 120.65 0)
-			(hide yes)
-			(show_name no)
-			(do_not_autoplace no)
-			(effects
-				(font
-					(size 1.27 1.27)
-				)
-			)
-		)
-		(pin "1"
-		)
-		(pin "A"
-		)
-		(pin "7"
-		)
-		(pin "8"
-		)
-		(pin "6"
-		)
-		(pin "2"
-		)
-		(pin "LHDP"
-		)
-		(pin "RHDP"
-		)
-		(pin "9"
-		)
-		(pin "4"
-		)
-		(pin "3"
-		)
-		(pin "5"
-		)
-		(pin "0"
-		)
-		(instances
-			(project "nixie-clock"
-				(path "/ee289ad4-b0b5-4cd2-aa28-bc5cdbd02292"
-					(reference "N1")
-					(unit 1)
-				)
-			)
-		)
 	)
 	(symbol

Commit message: work = force * distance
Other:
- sheet HV & Drivers renamed Power
- added sheet Tube Shift Registers (shift_registers.kicad_sch)
Changed lines of the file:
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@@
+	)
+	(sheet
+		(at 335.28 111.76)
+		(size 27.94 15.24)
+		(exclude_from_sim no)
+		(in_bom yes)
+		(on_board yes)
+		(dnp no)
+		(fields_autoplaced yes)
+		(stroke
+			(width 0.1524)
+			(type solid)
+		)
+		(fill
+			(color 0 0 0 0)
+		)
+		(property "Sheetname" "Tube Shift Registers"
+			(at 335.28 111.0484 0)
+			(show_name no)
+			(do_not_autoplace no)
+			(effects
+				(font
+					(size 1.27 1.27)
+				)
+				(justify left bottom)
+			)
+		)
+		(property "Sheetfile" "shift_registers.kicad_sch"
+			(at 335.28 127.5846 0)
+			(show_name no)
+			(do_not_autoplace no)
+			(effects
+				(font
+					(size 1.27 1.27)
+				)
+				(justify left top)
+			)
+		)
+		(pin "DCLK" input
+			(at 335.28 115.57 180)
+			(effects
+				(font
+					(size 1.27 1.27)
+				)
+				(justify left)
+			)
+		)
+		(pin "RCLK" input
+			(at 335.28 118.11 180)
+			(effects
+				(font
+					(size 1.27 1.27)
+				)
+				(justify left)
+			)
+		)
+		(pin "SDATA" input
+			(at 335.28 120.65 180)
+			(effects
+				(font
+					(size 1.27 1.27)
+				)
+				(justify left)
+			)
+		)
+		(pin "~{OE}" input
+			(at 335.28 123.19 180)
+			(effects
+				(font
+					(size 1.27 1.27)
+				)
+				(justify left)
+			)
+		)
+		(instances
+			(project "nixie-clock"
+				(path "/ee289ad4-b0b5-4cd2-aa28-bc5cdbd02292"
+					(page "10")
+				)
+			)
+		)
 	)
 	(sheet
@@
 			(color 0 0 0 0)
 		)
-		(property "Sheetname" "HV & Drivers"
+		(property "Sheetname" "Power"
 			(at 289.56 158.0384 0)
 			(show_name no)

Commit message: w
Parts:
- C1: value 1μF -> 22μF; Manufacturer Part Number CL31B105KAHNNNE -> (none); Vendor Part Number 1276-1097-1-ND -> (none)
- U2: Manufacturer Part Number ESP32-S3-WROOM-1-N4 -> ESP32-S3-WROOM-1-N8R8; Vendor Part Number 1965-ESP32-S3-WROOM-1-N4CT-ND -> 5407-ESP32-S3-WROOM-1-N8R8CT-ND
Connections:
- net +3.3V: now also U1.3 (ADCIN2)
Other:
- note added: "I2C ADDR:"
- note added: "I2C ADDR: 0x44, 0x45, 0x46"
- note added: "I2C ADDR: 0xD0"
- moved on the sheet: C14
Changed lines of the file:
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@@
 		(rev "1.0")
 	)
+	(text "I2C ADDR: 0x44, 0x45, 0x46"
+		(exclude_from_sim no)
+		(at 218.186 195.072 0)
+		(effects
+			(font
+				(size 1.27 1.27)
+			)
+		)
+	)
+	(text "I2C ADDR: 0xD0"
+		(exclude_from_sim no)
+		(at 171.196 199.644 0)
+		(effects
+			(font
+				(size 1.27 1.27)
+			)
+		)
+	)
+	(text "I2C ADDR:"
+		(exclude_from_sim no)
+		(at 203.2 122.682 0)
+		(effects
+			(font
+				(size 1.27 1.27)
+			)
+		)
+	)
 	(junction
 		(at 219.71 86.36)
@@
 	)
 	(junction
-		(at 314.96 67.31)
-		(diameter 0)
-		(color 0 0 0 0)
-	)
-	(junction
 		(at 186.69 163.83)
 		(diameter 0)
@@
 	)
 	(junction
+		(at 314.96 54.61)
+		(diameter 0)
+		(color 0 0 0 0)
+	)
+	(junction
 		(at 111.76 105.41)
 		(diameter 0)
@@
 	)
 	(junction
+		(at 148.59 116.84)
+		(diameter 0)
+		(color 0 0 0 0)
+	)
+	(junction
 		(at 121.92 91.44)
 		(diameter 0)
@@
 	)
 	(junction
-		(at 314.96 54.61)
+		(at 314.96 67.31)
 		(diameter 0)
 		(color 0 0 0 0)
@@
 	(wire
 		(pts
+			(xy 321.31 120.65) (xy 330.2 120.65)
+		)
+		(stroke
+			(width 0)
+			(type default)
+		)
+	)
+	(wire
+		(pts
 			(xy 208.28 86.36) (xy 208.28 88.9)
 		)
@@
 	(wire
 		(pts
-			(xy 325.12 54.61) (xy 314.96 54.61)
+			(xy 326.39 54.61) (xy 314.96 54.61)
 		)
 		(stroke
@@
 	(wire
 		(pts
-			(xy 325.12 54.61) (xy 325.12 57.15)
+			(xy 326.39 54.61) (xy 326.39 57.15)
 		)
 		(stroke
@@
 	(wire
 		(pts
+			(xy 276.86 93.98) (xy 281.94 93.98)
+		)
+		(stroke
+			(width 0)
+			(type default)
+		)
+	)
+	(wire
+		(pts
 			(xy 262.89 83.82) (xy 262.89 87.63)
 		)
@@
 	(wire
 		(pts
+			(xy 321.31 128.27) (xy 330.2 128.27)
+		)
+		(stroke
+			(width 0)
+			(type default)
+		)
+	)
+	(wire
+		(pts
 			(xy 121.92 91.44) (xy 144.78 91.44)
 		)
@@
 	(wire
 		(pts
+			(xy 148.59 116.84) (xy 153.67 116.84)
+		)
+		(stroke
+			(width 0)
+			(type default)
+		)
+	)
+	(wire
+		(pts
 			(xy 90.17 127) (xy 90.17 129.54)
 		)
@@
 	(wire
 		(pts
+			(xy 148.59 124.46) (xy 148.59 116.84)
+		)
+		(stroke
+			(width 0)
+			(type default)
+		)
+	)
+	(wire
+		(pts
+			(xy 276.86 88.9) (xy 281.94 88.9)
+		)
+		(stroke
+			(width 0)
+			(type default)
+		)
+	)
+	(wire
+		(pts
 			(xy 134.62 93.98) (xy 142.24 93.98)
 		)
@@
 	(wire
 		(pts
-			(xy 314.96 67.31) (xy 325.12 67.31)
+			(xy 314.96 67.31) (xy 326.39 67.31)
 		)
 		(stroke
@@
 	(wire
 		(pts
-			(xy 325.12 64.77) (xy 325.12 67.31)
+			(xy 326.39 64.77) (xy 326.39 67.31)
 		)
 		(stroke
@@
 	(wire
 		(pts
+			(xy 276.86 96.52) (xy 281.94 96.52)
+		)
+		(stroke
+			(width 0)
+			(type default)
+		)
+	)
+	(wire
+		(pts
 			(xy 219.71 86.36) (xy 219.71 88.9)
 		)
@@
 	(wire
 		(pts
-			(xy 139.7 116.84) (xy 153.67 116.84)
+			(xy 139.7 116.84) (xy 148.59 116.84)
+		)
+		(stroke
+			(width 0)
+			(type default)
+		)
+	)
+	(wire
+		(pts
+			(xy 153.67 124.46) (xy 148.59 124.46)
 		)
 		(stroke
@@
 	(wire
 		(pts
+			(xy 321.31 118.11) (xy 330.2 118.11)
+		)
+		(stroke
+			(width 0)
+			(type default)
+		)
+	)
+	(wire
+		(pts
 			(xy 109.22 93.98) (xy 134.62 93.98)
 		)
@@
 	(wire
 		(pts
+			(xy 321.31 125.73) (xy 330.2 125.73)
+		)
+		(stroke
+			(width 0)
+			(type default)
+		)
+	)
+	(wire
+		(pts
 			(xy 111.76 101.6) (xy 111.76 100.33)
 		)
@@
 	(wire
 		(pts
+			(xy 276.86 127) (xy 281.94 127)
+		)
+		(stroke
+			(width 0)
+			(type default)
+		)
+	)
+	(wire
+		(pts
 			(xy 234.95 168.91) (xy 234.95 171.45)
 		)
@@
 		)
 	)
+	(label "JTCK"
+		(at 330.2 118.11 180)
+		(effects
+			(font
+				(size 1.27 1.27)
+			)
+			(justify right bottom)
+		)
+	)
 	(label "~{INT}"
 		(at 186.69 179.07 180)
@@
 		)
 	)
+	(label "JTMS"
+		(at 330.2 128.27 180)
+		(effects
+			(font
+				(size 1.27 1.27)
+			)
+			(justify right bottom)
+		)
+	)
 	(label "SDA"
 		(at 198.12 176.53 0)
@@
 		)
 	)
+	(label "JTDI"
+		(at 330.2 125.73 180)
+		(effects
+			(font
+				(size 1.27 1.27)
+			)
+			(justify right bottom)
+		)
+	)
 	(label "SCL"
 		(at 198.12 173.99 0)
@@
 		)
 	)
+	(label "JTDO"
+		(at 330.2 120.65 180)
+		(effects
+			(font
+				(size 1.27 1.27)
+			)
+			(justify right bottom)
+		)
+	)
 	(symbol
 		(lib_id "Device:C")
@@
 	(symbol
 		(lib_id "Device:C")
-		(at 325.12 60.96 0)
+		(at 326.39 60.96 0)
 		(unit 1)
 		(body_style 1)
@@
 		(fields_autoplaced yes)
 		(property "Reference" "C14"
-			(at 328.93 59.6899 0)
+			(at 330.2 59.6899 0)
 			(show_name no)
 			(do_not_autoplace no)
@@
 		)
 		(property "Value" "100nF"
-			(at 328.93 62.2299 0)
+			(at 330.2 62.2299 0)
 			(show_name no)
 			(do_not_autoplace no)
@@
 		)
 		(property "Footprint" "Capacitor_SMD:C_1206_3216Metric_Pad1.33x1.80mm_HandSolder"
-			(at 326.0852 64.77 0)
+			(at 327.3552 64.77 0)
 			(hide yes)
 			(show_name no)
@@
 		)
 		(property "Datasheet" ""
-			(at 325.12 60.96 0)
+			(at 326.39 60.96 0)
 			(hide yes)
 			(show_name no)
@@
 		)
 		(property "Description" "Unpolarized capacitor"
-			(at 325.12 60.96 0)
+			(at 326.39 60.96 0)
 			(hide yes)
 			(show_name no)
@@
 		)
 		(property "Manufacturer Part Number" "C1206C104K5RACTU"
-			(at 325.12 60.96 0)
+			(at 326.39 60.96 0)
 			(hide yes)
 			(show_name no)
@@
 		)
 		(property "Vendor" "Digi-Key"
-			(at 325.12 60.96 0)
+			(at 326.39 60.96 0)
 			(hide yes)
 			(show_name no)
@@
 		)
 		(property "Vendor Part Number" "399-C1206C104K5RACTUCT-ND"
-			(at 325.12 60.96 0)
+			(at 326.39 60.96 0)
 			(hide yes)
 			(show_name no)
@@
 			)
 		)
-		(property "Value" "1μF"
+		(property "Value" "22μF"
 			(at 318.77 62.2299 0)
 			(show_name no)
@@
 			)
 		)
-		(property "Manufacturer Part Number" "CL31B105KAHNNNE"
+		(property "Manufacturer Part Number" ""
 			(at 314.96 60.96 0)
 			(hide yes)
@@
 			)
 		)
-		(property "Vendor Part Number" "1276-1097-1-ND"
+		(property "Vendor Part Number" ""
 			(at 314.96 60.96 0)
 			(hide yes)
@@
 			)
 		)
-		(property "Manufacturer Part Number" "ESP32-S3-WROOM-1-N4"
+		(property "Manufacturer Part Number" "ESP32-S3-WROOM-1-N8R8"
 			(at 297.18 106.68 0)
 			(hide yes)
@@
 			)
 		)
-		(property "Vendor Part Number" "1965-ESP32-S3-WROOM-1-N4CT-ND"
+		(property "Vendor Part Number" "5407-ESP32-S3-WROOM-1-N8R8CT-ND"
 			(at 297.18 106.68 0)
 			(hide yes)

Commit message: fix
Parts:
- added C35: 100nF, Capacitor_SMD:C_1206_3216Metric_Pad1.33x1.80mm_HandSolder, symbol Device:C
- added C36, C37: 22μF, Capacitor_SMD:C_1206_3216Metric_Pad1.33x1.80mm_HandSolder, symbol Device:C
- added J2: ESP Flash, symbol Connector_Generic:Conn_02x03_Odd_Even
- added J3: JTAG, symbol Connector_Generic:Conn_02x05_Odd_Even
- added L3: 4.7μH, symbol Device:L
- added R103, R4, R5: 10kΩ, Resistor_SMD:R_1206_3216Metric_Pad1.30x1.75mm_HandSolder, symbol Device:R_US
- added R104, R105: 4.7kΩ, Resistor_SMD:R_1206_3216Metric_Pad1.30x1.75mm_HandSolder, symbol Device:R_US
- added R106: 27kΩ, Resistor_SMD:R_1206_3216Metric_Pad1.30x1.75mm_HandSolder, symbol Device:R_US
- added R107: 13kΩ, Resistor_SMD:R_1206_3216Metric_Pad1.30x1.75mm_HandSolder, symbol Device:R_US
- added R108: 68kΩ, Resistor_SMD:R_1206_3216Metric_Pad1.30x1.75mm_HandSolder, symbol Device:R_US
- added R109: 3.3kΩ, Resistor_SMD:R_1206_3216Metric_Pad1.30x1.75mm_HandSolder, symbol Device:R_US
- added U30: AP63203WU, Package_TO_SOT_SMD:TSOT-23-6, symbol Regulator_Switching:AP63203WU
Connections:
- net +3.3V: now also C36.2, C37.2, J2.2 (Pin_2), J3.1 (Pin_1), L3.2, R104.1, R105.1, R4.1, U30.1 (FB); no longer C8.2, U1.1 (LDO_3V3), U1.3 (ADCIN2)
- net GND: now also C36.1, C37.1, J2.4 (Pin_4), J3.3 (Pin_3), J3.5 (Pin_5), J3.7 (Pin_7), J3.9 (Pin_9), R103.2, R107.2, R109.2, R5.2, U30.4 (GND)
- net JTCK: now also U2.32 (IO39), J3.4 (Pin_4)
- net JTDI: now also U2.34 (IO41), J3.8 (Pin_8)
- net JTDO: now also U2.33 (IO40), J3.6 (Pin_6)
- net JTMS: now also U2.35 (IO42), J3.2 (Pin_2)
- net SCL: now also U2.4 (IO4), R105.2
- net SDA: now also U2.5 (IO5), R104.2
- net Tube Shift Registers/DCLK: now also U2.7 (IO7)
- net Tube Shift Registers/RCLK: now also U2.12 (IO8)
- net Tube Shift Registers/SDATA: now also U2.17 (IO9)
- net Tube Shift Registers/~{OE}: now also U2.18 (IO10)
- net ~{INT}: now also U2.6 (IO6)
- net at C6.2, J1.A4 (VBUS), J1.A9 (VBUS)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: now also U30.2 (EN), U30.3 (IN)
- net ESP_EN: now reaches C5.1, R1.2, SW1.2, U2.3 (EN)
- net ESP_EN: now also J2.1 (Pin_1)
- net at U2.16 (IO46): now also R103.1
- net PWM_IN_1: now reaches U2.19 (IO11)
- net PWM_IN_2: now reaches U2.20 (IO12)
- net PWM_IN_3: now reaches U2.21 (IO13)
- net PWM_IN_4: now reaches U2.22 (IO14)
- net at U2.26 (IO45): now also R5.1
- net IO_0: now reaches U2.27 (IO0)
- net IO_0: now also J2.6 (Pin_6), R4.2
- net RXD_0: now reaches U2.36 (RXD0)
- net RXD_0: now also J2.5 (Pin_5)
- net TXD_0: now reaches U2.37 (TXD0)
- net TXD_0: now also J2.3 (Pin_3)
- net PWM_IN_5: now reaches U2.8 (IO15)
- net PWM_IN_6: now reaches U2.9 (IO16)
- net at U1.15 (DRAIN): now also U1.30 (DRAIN), U1.40 (DRAIN)
- net ADCIN1: now reaches U1.2 (ADCIN1)
- net ADCIN1: now also R106.2, R107.1
- net ADCIN3: now reaches U1.5 (ADCIN3)
- net ADCIN3: now also R108.2, R109.1
- net LDO_3.3V: now reaches U1.7 (ADCIN4)
- net LDO_3.3V: now also C8.2, U1.1 (LDO_3V3), U1.3 (ADCIN2), R106.1, R108.1
- new net: C35.1, U30.6 (BST)
- new net: C35.2, L3.1, U30.5 (SW)
- no-connect marks 3 -> 11
Other:
- added sheet Radio (radio.kicad_sch)
- sheet Tube Shift Registers ports: added PWM_IN_[1..6]; removed none
- moved on the sheet: C1, C14, C5, C8, R1, SW1, U2

Commit message: w
Parts:
- added C38, C39: 22μF, Capacitor_SMD:C_1206_3216Metric_Pad1.33x1.80mm_HandSolder, symbol Device:C
- added C40, C41: 10nF, Capacitor_SMD:C_1206_3216Metric_Pad1.33x1.80mm_HandSolder, symbol Device:C
- added C42: 10μF, Capacitor_SMD:C_1206_3216Metric_Pad1.33x1.80mm_HandSolder, symbol Device:C
- added C43: 100nF, Capacitor_SMD:C_1206_3216Metric_Pad1.33x1.80mm_HandSolder, symbol Device:C
- C6: value 10μF -> 10nF; Manufacturer Part Number CL31A106MAHNNNE -> (none); Vendor Part Number 1276-1181-1-ND -> (none)
- C9: value 47μF -> 10nF
Connections:
- net GND: now also C38.1, C39.1, C40.1, C41.1, C42.2, C43.2
- net VBUS: now also C38.2, C39.2; no longer C9.2
- net at C7.2, U1.32 (VBUS): now also C6.2, C9.2, J1.A4 (VBUS), J1.A9 (VBUS), J1.B4 (VBUS), J1.B9 (VBUS), U1.23 (VBUS_IN), U30.2 (EN), U30.3 (IN), C40.2, C41.2, C42.1, C43.1
Other:
- sheet Radio ports: added SCL, SDA; removed none
- moved on the sheet: C10, J1

Commit message: w
Connections:
- net ~{INT} renamed ~{RTC_INT}
Other:
- sheet Radio ports: added ~{RADIO_RST}; removed none
Changed lines of the file:
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@@
 		)
 	)
-	(label "~{INT}"
+	(label "~{RTC_INT}"
 		(at 186.69 179.07 180)
 		(effects
@@
 		)
 	)
-	(label "~{INT}"
+	(label "~{RTC_INT}"
 		(at 316.23 95.25 0)
 		(effects
@@
 			)
 		)
+		(pin "~{RADIO_RST}" input
+			(at 321.31 194.31 0)
+			(effects
+				(font
+					(size 1.27 1.27)
+				)
+				(justify right)
+			)
+		)

Commit message: w
Connections:
- net ~{FAULT_IN}: now reaches U1.18 (~{FAULT_IN})
- net CAP_MIS: now reaches U1.6 (CAP_MIS)
Other:
- sheet Power ports: added ~{HVDC_EN}; removed none
- sheet Radio ports: added ~{AUDIO_OUT_EN}; removed none
Changed lines of the file:
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@@
 	)
 	(junction
+		(at 209.55 111.76)
+		(diameter 0)
+		(color 0 0 0 0)
+	)
+	(junction
 		(at 186.69 26.67)
 		(diameter 0)
@@
 	(wire
 		(pts
-			(xy 316.23 85.09) (xy 321.31 85.09)
+			(xy 313.69 85.09) (xy 321.31 85.09)
 		)
 		(stroke
@@
 	(wire
 		(pts
+			(xy 209.55 111.76) (xy 222.25 111.76)
+		)
+		(stroke
+			(width 0)
+			(type default)
+		)
+	)
+	(wire
+		(pts
 			(xy 236.22 82.55) (xy 236.22 86.36)
 		)
@@
 	(wire
 		(pts
-			(xy 316.23 87.63) (xy 321.31 87.63)
+			(xy 313.69 87.63) (xy 321.31 87.63)
 		)
 		(stroke
@@
 	(wire
 		(pts
-			(xy 321.31 95.25) (xy 316.23 95.25)
+			(xy 313.69 95.25) (xy 321.31 95.25)
 		)
 		(stroke
@@
 	(wire
 		(pts
-			(xy 184.15 116.84) (xy 190.5 116.84)
-		)
-		(stroke
-			(width 0)
-			(type default)
-		)
-	)
-	(wire
-		(pts
 			(xy 138.43 124.46) (xy 138.43 116.84)
 		)
@@
 	(wire
 		(pts
-			(xy 316.23 80.01) (xy 321.31 80.01)
+			(xy 313.69 80.01) (xy 321.31 80.01)
 		)
 		(stroke
@@
 	(wire
 		(pts
+			(xy 321.31 196.85) (xy 336.55 196.85)
+		)
+		(stroke
+			(width 0)
+			(type default)
+		)
+	)
+	(wire
+		(pts
 			(xy 161.29 29.21) (xy 161.29 36.83)
 		)
@@
 	(wire
 		(pts
+			(xy 184.15 119.38) (xy 193.04 119.38)
+		)
+		(stroke
+			(width 0)
+			(type default)
+		)
+	)
+	(wire
+		(pts
 			(xy 121.92 104.14) (xy 121.92 107.95)
 		)
@@
 	(wire
 		(pts
+			(xy 184.15 96.52) (xy 193.04 96.52)
+		)
+		(stroke
+			(width 0)
+			(type default)
+		)
+	)
+	(wire
+		(pts
 			(xy 309.88 110.49) (xy 321.31 110.49)
 		)
@@
 	(wire
 		(pts
-			(xy 321.31 90.17) (xy 316.23 90.17)
+			(xy 313.69 90.17) (xy 321.31 90.17)
 		)
 		(stroke
@@
 	(wire
 		(pts
+			(xy 209.55 111.76) (xy 209.55 116.84)
+		)
+		(stroke
+			(width 0)
+			(type default)
+		)
+	)
+	(wire
+		(pts
 			(xy 118.11 36.83) (xy 118.11 39.37)
 		)
@@
 	(wire
 		(pts
+			(xy 313.69 82.55) (xy 321.31 82.55)
+		)
+		(stroke
+			(width 0)
+			(type default)
+		)
+	)
+	(wire
+		(pts
 			(xy 138.43 73.66) (xy 138.43 76.2)
 		)
@@
 	(wire
 		(pts
-			(xy 321.31 92.71) (xy 316.23 92.71)
+			(xy 313.69 92.71) (xy 321.31 92.71)
 		)
 		(stroke
@@
 	(wire
 		(pts
+			(xy 184.15 111.76) (xy 209.55 111.76)
+		)
+		(stroke
+			(width 0)
+			(type default)
+		)
+	)
+	(wire
+		(pts
 			(xy 184.15 127) (xy 187.96 127)
 		)
@@
 	(wire
 		(pts
+			(xy 184.15 116.84) (xy 193.04 116.84)
+		)
+		(stroke
+			(width 0)
+			(type default)
+		)
+	)
+	(wire
+		(pts
 			(xy 302.26 72.39) (xy 302.26 74.93)
 		)
@@
 	(wire
 		(pts
-			(xy 184.15 119.38) (xy 190.5 119.38)
+			(xy 309.88 118.11) (xy 321.31 118.11)
 		)
 		(stroke
@@
 	(wire
 		(pts
-			(xy 309.88 118.11) (xy 321.31 118.11)
+			(xy 346.71 179.07) (xy 349.25 179.07)
 		)
 		(stroke
@@
 	(wire
 		(pts
-			(xy 346.71 179.07) (xy 349.25 179.07)
+			(xy 351.79 77.47) (xy 359.41 77.47)
 		)
 		(stroke
@@
 	(wire
 		(pts
-			(xy 351.79 77.47) (xy 359.41 77.47)
+			(xy 138.43 124.46) (xy 138.43 129.54)
 		)
 		(stroke
@@
 	(wire
 		(pts
-			(xy 138.43 124.46) (xy 138.43 129.54)
+			(xy 351.79 107.95) (xy 359.41 107.95)
 		)
 		(stroke
@@
 	(wire
 		(pts
-			(xy 351.79 107.95) (xy 359.41 107.95)
+			(xy 146.05 121.92) (xy 153.67 121.92)
 		)
 		(stroke
@@
 	(wire
 		(pts
-			(xy 146.05 121.92) (xy 153.67 121.92)
+			(xy 351.79 120.65) (xy 359.41 120.65)
+		)
+		(stroke
+			(width 0)
+			(type default)
+		)
+	)
+	(wire
+		(pts
+			(xy 322.58 168.91) (xy 332.74 168.91)
 		)
 		(stroke
@@
 	(wire
 		(pts
+			(xy 321.31 194.31) (xy 336.55 194.31)
+		)
+		(stroke
+			(width 0)
+			(type default)
+		)
+	)
+	(wire
+		(pts
 			(xy 234.95 168.91) (xy 234.95 171.45)
 		)
@@
 	(wire
 		(pts
+			(xy 351.79 118.11) (xy 359.41 118.11)
+		)
+		(stroke
+			(width 0)
+			(type default)
+		)
+	)
+	(wire
+		(pts
 			(xy 161.29 36.83) (xy 163.83 36.83)
 		)
@@
 		)
 	)
+	(label "~{RADIO_RST}"
+		(at 336.55 194.31 180)
+		(effects
+			(font
+				(size 1.27 1.27)
+			)
+			(justify right bottom)
+		)
+	)
 	(label "ESP_EN"
 		(at 320.04 74.93 180)
@@
 		)
 	)
+	(label "CAP_MIS"
+		(at 369.57 86.36 180)
+		(effects
+			(font
+				(size 1.27 1.27)
+			)
+			(justify right bottom)
+		)
+	)
 	(label "SDA"
 		(at 146.05 173.99 0)
@@
 	)
 	(label "SDA"
-		(at 190.5 119.38 180)
+		(at 193.04 119.38 180)
 		(effects
 			(font
@@
 		)
 	)
+	(label "~{HVDC_EN}"
+		(at 369.57 97.79 180)
+		(effects
+			(font
+				(size 1.27 1.27)
+			)
+			(justify right bottom)
+		)
+	)
 	(label "PWM_IN_5"
 		(at 320.04 118.11 180)
@@
 	)
 	(label "SCL"
-		(at 190.5 116.84 180)
+		(at 193.04 116.84 180)
+		(effects
+			(font
+				(size 1.27 1.27)
+			)
+			(justify right bottom)
+		)
+	)
+	(label "CAP_MIS"
+		(at 193.04 96.52 180)
 		(effects
 			(font
@@
 		)
 	)
+	(label "~{HVDC_EN}"
+		(at 332.74 168.91 180)
+		(effects
+			(font
+				(size 1.27 1.27)
+			)
+			(justify right bottom)
+		)
+	)
 	(label "SDA"
-		(at 316.23 92.71 0)
+		(at 313.69 92.71 0)
 		(effects
 			(font
@@
 		)
 	)
+	(label "~{FAULT_IN}"
+		(at 369.57 101.6 180)
+		(effects
+			(font
+				(size 1.27 1.27)
+			)
+			(justify right bottom)
+		)
+	)
 	(label "D-"
 		(at 90.17 100.33 180)
@@
 		)
 	)
+	(label "~{RADIO_RST}"
+		(at 369.57 91.44 180)
+		(effects
+			(font
+				(size 1.27 1.27)
+			)
+			(justify right bottom)
+		)
+	)
 	(label "SCL"
-		(at 316.23 90.17 0)
+		(at 313.69 90.17 0)
 		(effects
 			(font
@@
 		)
 	)
+	(label "~{AUDIO_OUT_EN}"
+		(at 369.57 95.25 180)
+		(effects
+			(font
+				(size 1.27 1.27)
+			)
+			(justify right bottom)
+		)
+	)
 	(label "IO_0"
 		(at 318.77 57.15 90)
@@
 		)
 	)
+	(label "~{FAULT_IN}"
+		(at 222.25 111.76 180)
+		(effects
+			(font
+				(size 1.27 1.27)
+			)
+			(justify right bottom)
+		)
+	)
 	(label "JTDI"
 		(at 359.41 107.95 180)
@@
 		)
 	)
+	(label "~{AUDIO_OUT_EN}"
+		(at 336.55 196.85 180)
+		(effects
+			(font
+				(size 1.27 1.27)
+			)
+			(justify right bottom)
+		)
+	)
 	(label "LDO_3.3V"
 		(at 90.17 140.97 270)
@@
 	)
 	(label "~{RTC_INT}"
-		(at 316.23 95.25 0)
+		(at 313.69 95.25 0)
 		(effects
 			(font
@@
 	)
 	(label "IO_0"
-		(at 316.23 80.01 0)
+		(at 313.69 80.01 0)
 		(effects
 			(font
@@
 			)
 		)
+		(pin "~{HVDC_EN}" input
+			(at 322.58 168.91 0)
+			(effects
+				(font
+					(size 1.27 1.27)
+				)
+				(justify right)
+			)
+		)
 		(instances
 			(project "nixie-clock"
@@
 			(effects
 				(font
+					(size 1.27 1.27)
+				)
+				(justify right)
+			)
+		)
+		(pin "~{AUDIO_OUT_EN}" input
+			(at 321.31 196.85 0)
+			(effects
+				(font
