File: pcb/nixie-clock.kicad_sch (KiCad schematic)
At the start: 45 parts, among them J1 USB_C_Receptacle, J2 ESP Flash, J3 JTAG, SW1 Reset, U1 TPS25730D, U2 ESP32-S3-WROOM-1, U3 DS3231MZ, U30 AP63203WU, U4 STS4X

Commit message: w
Parts:
- added R129: 1kΩ, Resistor_SMD:R_1206_3216Metric_Pad1.30x1.75mm_HandSolder, symbol Device:R_US
Connections:
- net +3.3V: now also R129.2
- net CAP_MIS: now also U2.24 (IO47)
- net ~{AUDIO_OUT_EN}: now also U2.38 (IO2)
- net ~{FAULT_IN}: now also U2.25 (IO48), R129.1
- net ~{HVDC_EN}: now also U2.15 (IO3)
- net ~{RADIO_RST}: now also U2.39 (IO1)
- no-connect marks 11 -> 15
Other:
- moved on the sheet: C5, R1, SW1

Commit message: w
Parts:
- BT1: footprint (none) -> Battery:BatteryHolder_MPD_BC2003_1x2032
- C10, C11, C42, C8: Manufacturer Part Number CL31A106MAHNNNE -> (none); Vendor Part Number 1276-1181-1-ND -> (none)
- C14, C15, C16, C43, C5: Manufacturer Part Number C1206C104K5RACTU -> (none); Vendor Part Number 399-C1206C104K5RACTUCT-ND -> (none)
- C2, C3: Manufacturer Part Number CL31B105KAHNNNE -> (none); Vendor Part Number 1276-1097-1-ND -> (none)
- C7: Manufacturer Part Number CL31B475KAHNNNE -> (none); Vendor Part Number 1276-1055-1-ND -> (none)
- J2: footprint (none) -> Connector_IDC:IDC-Header_2x03_P2.54mm_Vertical
- J3: footprint (none) -> Connector_IDC:IDC-Header_2x05_P2.54mm_Vertical
- L3: footprint (none) -> Inductor_SMD:L_0603_1608Metric_Pad1.05x0.95mm_HandSolder; Manufacturer Part Number (none) -> LQM18PN4R7MFRL; Vendor (none) -> Digi-Key; Vendor Part Number (none) -> 490-12065-1-ND
- R1, R103, R104, R105, R106, R107, R108, R109, R129, R4, R5: Manufacturer Part Number RMCF1206FT10K0 -> (none); Vendor Part Number RMCF1206FT10K0CT-ND -> (none)
Changed lines of the file:
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@@
 			)
 		)
-		(property "Manufacturer Part Number" "CL31B475KAHNNNE"
+		(property "Manufacturer Part Number" ""
 			(at 149.86 80.01 0)
 			(hide yes)
@@
 			)
 		)
-		(property "Vendor Part Number" "1276-1055-1-ND"
+		(property "Vendor Part Number" ""
 			(at 149.86 80.01 0)
 			(hide yes)
@@
 			)
 		)
-		(property "Manufacturer Part Number" "C1206C104K5RACTU"
+		(property "Manufacturer Part Number" ""
 			(at 365.76 52.07 0)
 			(hide yes)
@@
 			)
 		)
-		(property "Vendor Part Number" "399-C1206C104K5RACTUCT-ND"
+		(property "Vendor Part Number" ""
 			(at 365.76 52.07 0)
 			(hide yes)
@@
 			)
 		)
-		(property "Manufacturer Part Number" "C1206C104K5RACTU"
+		(property "Manufacturer Part Number" ""
 			(at 118.11 33.02 0)
 			(hide yes)
@@
 			)
 		)
-		(property "Vendor Part Number" "399-C1206C104K5RACTUCT-ND"
+		(property "Vendor Part Number" ""
 			(at 118.11 33.02 0)
 			(hide yes)
@@
 			)
 		)
-		(property "Manufacturer Part Number" "RMCF1206FT10K0"
+		(property "Manufacturer Part Number" ""
 			(at 318.77 46.99 0)
 			(hide yes)
@@
 			)
 		)
-		(property "Vendor Part Number" "RMCF1206FT10K0CT-ND"
+		(property "Vendor Part Number" ""
 			(at 318.77 46.99 0)
 			(hide yes)
@@
 			)
 		)
-		(property "Manufacturer Part Number" "RMCF1206FT10K0"
+		(property "Manufacturer Part Number" ""
 			(at 73.66 171.45 0)
 			(hide yes)
@@
 			)
 		)
-		(property "Vendor Part Number" "RMCF1206FT10K0CT-ND"
+		(property "Vendor Part Number" ""
 			(at 73.66 171.45 0)
 			(hide yes)
@@
 			)
 		)
-		(property "Manufacturer Part Number" "RMCF1206FT10K0"
+		(property "Manufacturer Part Number" ""
 			(at 369.57 123.19 0)
 			(hide yes)
@@
 			)
 		)
-		(property "Vendor Part Number" "RMCF1206FT10K0CT-ND"
+		(property "Vendor Part Number" ""
 			(at 369.57 123.19 0)
 			(hide yes)
@@
 			)
 		)
-		(property "Manufacturer Part Number" "RMCF1206FT10K0"
+		(property "Manufacturer Part Number" ""
 			(at 394.97 91.44 0)
 			(hide yes)
@@
 			)
 		)
-		(property "Vendor Part Number" "RMCF1206FT10K0CT-ND"
+		(property "Vendor Part Number" ""
 			(at 394.97 91.44 0)
 			(hide yes)
@@
 			)
 		)
-		(property "Footprint" ""
+		(property "Footprint" "Connector_IDC:IDC-Header_2x03_P2.54mm_Vertical"
 			(at 354.33 199.39 0)
 			(hide yes)
@@
 			)
 		)
-		(property "Manufacturer Part Number" "C1206C104K5RACTU"
+		(property "Manufacturer Part Number" ""
 			(at 196.85 157.48 0)
 			(hide yes)
@@
 			)
 		)
-		(property "Vendor Part Number" "399-C1206C104K5RACTUCT-ND"
+		(property "Vendor Part Number" ""
 			(at 196.85 157.48 0)
 			(hide yes)
@@
 			)
 		)
-		(property "Manufacturer Part Number" "RMCF1206FT10K0"
+		(property "Manufacturer Part Number" ""
 			(at 90.17 171.45 0)
 			(hide yes)
@@
 			)
 		)
-		(property "Vendor Part Number" "RMCF1206FT10K0CT-ND"
+		(property "Vendor Part Number" ""
 			(at 90.17 171.45 0)
 			(hide yes)
@@
 			)
 		)
-		(property "Footprint" ""
+		(property "Footprint" "Connector_IDC:IDC-Header_2x05_P2.54mm_Vertical"
 			(at 354.33 173.99 0)
 			(hide yes)
@@
 			)
 		)
-		(property "Manufacturer Part Number" "RMCF1206FT10K0"
+		(property "Manufacturer Part Number" ""
 			(at 384.81 91.44 0)
 			(hide yes)
@@
 			)
 		)
-		(property "Vendor Part Number" "RMCF1206FT10K0CT-ND"
+		(property "Vendor Part Number" ""
 			(at 384.81 91.44 0)
 			(hide yes)
@@
 			)
 		)
-		(property "Manufacturer Part Number" "CL31A106MAHNNNE"
+		(property "Manufacturer Part Number" ""
 			(at 196.85 97.79 0)
 			(hide yes)
@@
 			)
 		)
-		(property "Vendor Part Number" "1276-1181-1-ND"
+		(property "Vendor Part Number" ""
 			(at 196.85 97.79 0)
 			(hide yes)
@@
 			)
 		)
-		(property "Manufacturer Part Number" "RMCF1206FT10K0"
+		(property "Manufacturer Part Number" ""
 			(at 379.73 123.19 0)
 			(hide yes)
@@
 			)
 		)
-		(property "Vendor Part Number" "RMCF1206FT10K0CT-ND"
+		(property "Vendor Part Number" ""
 			(at 379.73 123.19 0)
 			(hide yes)
@@
 			)
 		)
-		(property "Manufacturer Part Number" "RMCF1206FT10K0"
+		(property "Manufacturer Part Number" ""
 			(at 209.55 120.65 0)
 			(hide yes)
@@
 			)
 		)
-		(property "Vendor Part Number" "RMCF1206FT10K0CT-ND"
+		(property "Vendor Part Number" ""
 			(at 209.55 120.65 0)
 			(hide yes)
@@
 			)
 		)
-		(property "Manufacturer Part Number" "CL31B105KAHNNNE"
+		(property "Manufacturer Part Number" ""
 			(at 234.95 175.26 0)
 			(hide yes)
@@
 			)
 		)
-		(property "Vendor Part Number" "1276-1097-1-ND"
+		(property "Vendor Part Number" ""
 			(at 234.95 175.26 0)
 			(hide yes)
@@
 			)
 		)
-		(property "Manufacturer Part Number" "C1206C104K5RACTU"
+		(property "Manufacturer Part Number" ""
 			(at 245.11 175.26 0)
 			(hide yes)
@@
 			)
 		)
-		(property "Vendor Part Number" "399-C1206C104K5RACTUCT-ND"
+		(property "Vendor Part Number" ""
 			(at 245.11 175.26 0)
 			(hide yes)
@@
 			)
 		)
-		(property "Manufacturer Part Number" "CL31B105KAHNNNE"
+		(property "Manufacturer Part Number" ""
 			(at 186.69 157.48 0)
 			(hide yes)
@@
 			)
 		)
-		(property "Vendor Part Number" "1276-1097-1-ND"
+		(property "Vendor Part Number" ""
 			(at 186.69 157.48 0)
 			(hide yes)
@@
 			)
 		)
-		(property "Manufacturer Part Number" "RMCF1206FT10K0"
+		(property "Manufacturer Part Number" ""
 			(at 294.64 68.58 0)
 			(hide yes)
@@
 			)
 		)
-		(property "Vendor Part Number" "RMCF1206FT10K0CT-ND"
+		(property "Vendor Part Number" ""
 			(at 294.64 68.58 0)
 			(hide yes)
@@
 			)
 		)
-		(property "Footprint" ""
+		(property "Footprint" "Inductor_SMD:L_0603_1608Metric_Pad1.05x0.95mm_HandSolder"
 			(at 180.34 26.67 0)
 			(hide yes)
@@
 			)
 		)
+		(property "Manufacturer Part Number" "LQM18PN4R7MFRL"
+			(at 180.34 26.67 90)
+			(hide yes)
+			(show_name no)
+			(do_not_autoplace no)
+			(effects
+				(font
+					(size 1.27 1.27)
+				)
+			)
+		)
+		(property "Vendor" "Digi-Key"
+			(at 180.34 26.67 90)
+			(hide yes)
+			(show_name no)
+			(do_not_autoplace no)
+			(effects
+				(font
+					(size 1.27 1.27)
+				)
+			)
+		)
+		(property "Vendor Part Number" "490-12065-1-ND"
+			(at 180.34 26.67 90)
+			(hide yes)
+			(show_name no)
+			(do_not_autoplace no)
+			(effects
+				(font
+					(size 1.27 1.27)
+				)
+			)
+		)
 		(pin "2"
 		)
@@
 			)
 		)
-		(property "Manufacturer Part Number" "RMCF1206FT10K0"
+		(property "Manufacturer Part Number" ""
 			(at 90.17 156.21 0)
 			(hide yes)
@@
 			)
 		)
-		(property "Vendor Part Number" "RMCF1206FT10K0CT-ND"
+		(property "Vendor Part Number" ""
 			(at 90.17 156.21 0)
 			(hide yes)
@@
 			)
 		)
-		(property "Manufacturer Part Number" "CL31A106MAHNNNE"
+		(property "Manufacturer Part Number" ""
 			(at 138.43 135.89 0)
 			(hide yes)
@@
 			)
 		)
-		(property "Vendor Part Number" "1276-1181-1-ND"
+		(property "Vendor Part Number" ""
 			(at 138.43 135.89 0)
 			(hide yes)
@@
 			)
 		)
-		(property "Manufacturer Part Number" "RMCF1206FT10K0"
+		(property "Manufacturer Part Number" ""
 			(at 73.66 156.21 0)
 			(hide yes)
@@
 			)
 		)
-		(property "Vendor Part Number" "RMCF1206FT10K0CT-ND"
+		(property "Vendor Part Number" ""
 			(at 73.66 156.21 0)
 			(hide yes)
@@
 			)
 		)
-		(property "Footprint" ""
+		(property "Footprint" "Battery:BatteryHolder_MPD_BC2003_1x2032"
 			(at 129.54 171.196 90)
 			(hide yes)
@@
 			)
 		)
-		(property "Manufacturer Part Number" "CL31A106MAHNNNE"
+		(property "Manufacturer Part Number" ""
 			(at 236.22 92.71 0)
 			(hide yes)
@@
 			)
 		)
-		(property "Vendor Part Number" "1276-1181-1-ND"
+		(property "Vendor Part Number" ""
 			(at 236.22 92.71 0)
 			(hide yes)
@@
 			)
 		)
-		(property "Manufacturer Part Number" "CL31A106MAHNNNE"
+		(property "Manufacturer Part Number" ""
 			(at 106.68 33.02 0)
 			(hide yes)
@@
 			)
 		)
-		(property "Vendor Part Number" "1276-1181-1-ND"
+		(property "Vendor Part Number" ""
 			(at 106.68 33.02 0)
 			(hide yes)
@@
 			)
 		)
-		(property "Manufacturer Part Number" "C1206C104K5RACTU"
+		(property "Manufacturer Part Number" ""
 			(at 294.64 82.55 0)
 			(hide yes)
@@
 			)
 		)
-		(property "Vendor Part Number" "399-C1206C104K5RACTUCT-ND"
+		(property "Vendor Part Number" ""
 			(at 294.64 82.55 0)
 			(hide yes)
