File: pcb/nixie-clock.kicad_sch (KiCad schematic)
At the start: 46 parts, among them J1 USB_C_Receptacle, J2 ESP Flash, J3 JTAG, SW1 Reset, U1 TPS25730D, U2 ESP32-S3-WROOM-1, U3 DS3231MZ, U30 AP63203WU, U4 STS4X

Commit message: Update nixie-clock.kicad_sch
Connections:
- net ~{HVDC_EN}: no longer U2.15 (IO3)
Other:
- note added: "TODO check to see if IO3 and IO 45 & 46 need special treatment"
Changed lines of the file:
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@@
+		)
+	)
+	(text "TODO check to see if IO3 and IO 45 & 46 need special treatment"
+		(exclude_from_sim no)
+		(at 392.176 67.818 0)
+		(effects
+			(font
+				(size 1.27 1.27)
+			)
 		)
 	)
@@
 	(wire
 		(pts
+			(xy 302.26 87.63) (xy 317.5 87.63)
+		)
+		(stroke
+			(width 0)
+			(type default)
+		)
+	)
+	(wire
+		(pts
 			(xy 208.28 96.52) (xy 208.28 99.06)
 		)
@@
 		(pts
 			(xy 87.63 26.67) (xy 87.63 86.36)
-		)
-		(stroke
-			(width 0)
-			(type default)
-		)
-	)
-	(wire
-		(pts
-			(xy 306.07 87.63) (xy 321.31 87.63)
 		)
 		(stroke
@@
 		)
 	)
-	(label "~{HVDC_EN}"
-		(at 306.07 87.63 0)
-		(effects
-			(font
-				(size 1.27 1.27)
-			)
-			(justify left bottom)
-		)
-	)
 	(label "PWM_IN_5"
 		(at 320.04 118.11 180)
@@
 		(effects
 			(font
+				(size 1.27 1.27)
+			)
+			(justify left bottom)
+		)
+	)
+	(label "~{HVDC_EN}"
+		(at 302.26 87.63 0)
+		(effects
+			(font
