File: pcb/radio.kicad_sch (KiCad schematic)
At the start: 6 parts, among them U29 Si4735-D60-GU

Commit message: w
Parts:
- added J4: AM Antenna, symbol Connector:Conn_Coaxial
- added J5: FM Antenna, symbol Connector:Conn_Coaxial
Connections:
- net at D6.2 (VP), D6.3 (VN), L1.2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: now also J4.2 (Ext), J5.2 (Ext)
- net at C33.2, D6.1 (CH1): now also J5.1 (In)
- net at C34.2, L1.1: now also J4.1 (In)
Other:
- moved on the sheet: C33, C34, D6, L1, L2

Commit message: w
Parts:
- added C44, C45: 12.5pF, Capacitor_SMD:C_1206_3216Metric_Pad1.33x1.80mm_HandSolder, symbol Device:C
- added C46: 22nF, Capacitor_SMD:C_1206_3216Metric_Pad1.33x1.80mm_HandSolder, symbol Device:C
- added C47, C48, C51, C52: 22μF, Capacitor_SMD:C_1206_3216Metric_Pad1.33x1.80mm_HandSolder, symbol Device:C
- added C49, C50: 100nF, Capacitor_SMD:C_1206_3216Metric_Pad1.33x1.80mm_HandSolder, symbol Device:C
- added J6: AudioJack3_SwitchTR, symbol Connector_Audio:AudioJack3_SwitchTR
- added R110, R115, R116, R117, R118: 10kΩ, Resistor_SMD:R_1206_3216Metric_Pad1.30x1.75mm_HandSolder, symbol Device:R_US
- added R111, R113: 2.2kΩ, Resistor_SMD:R_1206_3216Metric_Pad1.30x1.75mm_HandSolder, symbol Device:R_US
- added R112, R114: 4.7kΩ, Resistor_SMD:R_1206_3216Metric_Pad1.30x1.75mm_HandSolder, symbol Device:R_US
- added U31: TDA1308, symbol Amplifier_Audio:TDA1308
- added Y1: 32.768kHz, symbol Device:Crystal
- C33, C34: Manufacturer Part Number C1206C104K5RACTU -> (none); Vendor Part Number 399-C1206C104K5RACTUCT-ND -> (none)
Connections:
- net +3.3V: now also C46.2, C49.2, R117.1, U31.8 (V+)
- net GND: now also D6.2 (VP), D6.3 (VN), J4.2 (Ext), J5.2 (Ext), L1.2, L2.2, U29.9 (RFGND), C44.1, C45.1, C49.1, C50.1, J6.S, R110.2, R115.2, R116.2, R118.2, U31.4 (VSS)
- net ~{RADIO_RST}: now reaches U29.15 (~{RST})
- net at U29.16 (~{SEN}): now also R110.1
- net XTAL2: now reaches U29.19 (RCLK)
- net XTAL2: now also C45.2, Y1.2
- net at U29.22 (DBYP): now also C46.1
- net ROUT: now reaches U29.23 (ROUT/[DOUT])
- net ROUT: now also C48.2
- net LOUT: now reaches U29.24 (LOUT/[DFS])
- net LOUT: now also C47.2
- net XTAL1: now reaches U29.3 (GPO3/[DCLK])
- net XTAL1: now also C44.2, Y1.1
- new net: R111.2, R112.1, U31.2 (-)
- new net: C51.2, R112.2, U31.1
- new net: C50.2, R117.2, R118.1, U31.3 (+), U31.5 (+)
- new net: R113.2, R114.1, U31.6 (-)
- new net: C52.2, R114.2, U31.7
- new net: C47.1, R113.1
- new net: C51.1, J6.T, R115.1
- new net: C48.1, R111.1
- new net: C52.1, J6.R, R116.1
- new net: J6.RN, J6.TN
- no-connect marks 0 -> 4
Other:
- moved on the sheet: C33, C34, D6, J4, J5, L1, L2, U29

Commit message: w
Parts:
- added U7: TS3A5223RSW, Package_DFN_QFN:Texas_RSW0010A_UQFN-10_1.4x1.8mm_P0.4mm, symbol Analog_Switch:TS3A5223RSW
Connections:
- net +3.3V: now also U7.1 (VCC)
- net GND: now also U7.6 (GND)
- net LOUT: now also C48.2; no longer C47.2
- net ROUT: now also C47.2; no longer C48.2
- net at C51.1, R115.1: now also U7.3; no longer J6.T
- net at C52.1, R116.1: now also U7.9; no longer J6.R
- new net: J6.T, U7.5
- new net: J6.R, U7.7
- new net ~{AUDIO_OUT_EN}: U7.4, U7.8
Other:
- moved on the sheet: C47, C48, C49, C50, C51, C52, J4, J5, J6, R111, R112, R113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

Commit message: w
Parts:
- J4, J5: footprint (none) -> Connector_Coaxial:BNC_TEConnectivity_1478204_Vertical
- J6: footprint (none) -> Connector_Audio:Jack_3.5mm_CUI_SJ1-3535NG_Horizontal
- Y1: footprint (none) -> Crystal:Crystal_SMD_3215-2Pin_3.2x1.5mm
Changed lines of the file:
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@@
 			)
 		)
-		(property "Footprint" ""
+		(property "Footprint" "Connector_Audio:Jack_3.5mm_CUI_SJ1-3535NG_Horizontal"
 			(at 345.44 128.27 0)
 			(hide yes)
@@
 			)
 		)
-		(property "Footprint" ""
+		(property "Footprint" "Connector_Coaxial:BNC_TEConnectivity_1478204_Vertical"
 			(at 182.88 74.93 0)
 			(hide yes)
@@
 			)
 		)
-		(property "Footprint" ""
+		(property "Footprint" "Crystal:Crystal_SMD_3215-2Pin_3.2x1.5mm"
 			(at 83.82 125.73 0)
 			(hide yes)
@@
 			)
 		)
-		(property "Footprint" ""
+		(property "Footprint" "Connector_Coaxial:BNC_TEConnectivity_1478204_Vertical"
 			(at 182.88 87.63 0)
 			(hide yes)

Commit message: w
Parts:
- added U8: PAM8908, Package_DFN_QFN:QFN-16-1EP_3x3mm_P0.5mm_EP1.7x1.7mm, symbol Amplifier_Audio:PAM8908
- C44, C45: Manufacturer Part Number C1206C104K5RACTU -> (none); Vendor Part Number 399-C1206C104K5RACTUCT-ND -> (none)
- R110, R115, R116, R117, R118: Manufacturer Part Number RMCF1206FT10K0 -> (none); Vendor Part Number RMCF1206FT10K0CT-ND -> (none)
Changed lines of the file:
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@@
 			)
 		)
-		(property "Manufacturer Part Number" "C1206C104K5RACTU"
+		(property "Manufacturer Part Number" ""
 			(at 76.2 133.35 0)
 			(hide yes)
@@
 			)
 		)
-		(property "Vendor Part Number" "399-C1206C104K5RACTUCT-ND"
+		(property "Vendor Part Number" ""
 			(at 76.2 133.35 0)
 			(hide yes)
@@
 			)
 		)
-		(property "Manufacturer Part Number" "RMCF1206FT10K0"
+		(property "Manufacturer Part Number" ""
 			(at 240.03 48.26 0)
 			(hide yes)
@@
 			)
 		)
-		(property "Vendor Part Number" "RMCF1206FT10K0CT-ND"
+		(property "Vendor Part Number" ""
 			(at 240.03 48.26 0)
 			(hide yes)
@@
 			)
 		)
-		(property "Manufacturer Part Number" "RMCF1206FT10K0"
+		(property "Manufacturer Part Number" ""
 			(at 240.03 125.73 0)
 			(hide yes)
@@
 			)
 		)
-		(property "Vendor Part Number" "RMCF1206FT10K0CT-ND"
+		(property "Vendor Part Number" ""
 			(at 240.03 125.73 0)
 			(hide yes)
@@
 			)
 		)
-		(property "Manufacturer Part Number" "RMCF1206FT10K0"
+		(property "Manufacturer Part Number" ""
 			(at 293.37 120.65 0)
 			(hide yes)
@@
 			)
 		)
-		(property "Vendor Part Number" "RMCF1206FT10K0CT-ND"
+		(property "Vendor Part Number" ""
 			(at 293.37 120.65 0)
 			(hide yes)
@@
 	)
 	(symbol
+		(lib_id "Amplifier_Audio:PAM8908")
+		(at 260.35 171.45 0)
+		(unit 1)
+		(body_style 1)
+		(exclude_from_sim no)
+		(in_bom yes)
+		(on_board yes)
+		(in_pos_files yes)
+		(dnp no)
+		(fields_autoplaced yes)
+		(property "Reference" "U8"
+			(at 262.4933 148.59 0)
+			(show_name no)
+			(do_not_autoplace no)
+			(effects
+				(font
+					(size 1.27 1.27)
+				)
+				(justify left)
+			)
+		)
+		(property "Value" "PAM8908"
+			(at 262.4933 151.13 0)
+			(show_name no)
+			(do_not_autoplace no)
+			(effects
+				(font
+					(size 1.27 1.27)
+				)
+				(justify left)
+			)
+		)
+		(property "Footprint" "Package_DFN_QFN:QFN-16-1EP_3x3mm_P0.5mm_EP1.7x1.7mm"
+			(at 264.16 190.5 0)
+			(hide yes)
+			(show_name no)
+			(do_not_autoplace no)
+			(effects
+				(font
+					(size 1.27 1.27)
+				)
+				(justify left)
+			)
+		)
+		(property "Datasheet" "https://www.diodes.com/datasheet/download/PAM8908.pdf"
+			(at 264.16 193.04 0)
+			(hide yes)
+			(show_name no)
+			(do_not_autoplace no)
+			(effects
+				(font
+					(size 1.27 1.27)
+				)
+				(justify left)
+			)
+		)
+		(property "Description" "60mW 2.5-5.5V differential stereo headphone amplifier with adjustable gain, QFN-16"
+			(at 264.16 195.58 0)
+			(hide yes)
+			(show_name no)
+			(do_not_autoplace no)
+			(effects
+				(font
+					(size 1.27 1.27)
+				)
+				(justify left)
+			)
+		)
+		(pin "1"
+		)
+		(pin "16"
+		)
+		(pin "15"
+		)
+		(pin "9"
+		)
+		(pin "5"
+		)
+		(pin "10"
+		)
+		(pin "3"
+		)
+		(pin "6"
+		)
+		(pin "2"
+		)
+		(pin "17"
+		)
+		(pin "14"
+		)
+		(pin "13"
+		)
+		(pin "8"
+		)
+		(pin "12"
+		)
+		(pin "7"
+		)
+		(pin "11"
+		)
+		(pin "4"
+		)
+		(instances
+			(project "nixie-clock"
+				(path "/ee289ad4-b0b5-4cd2-aa28-bc5cdbd02292/f8d3b7da-a2a9-47f4-8e07-f9acd571f3e8"
+					(reference "U8")
+					(unit 1)
+				)
+			)
+		)
+	)
+	(symbol
 		(lib_id "power:GND")
 		(at 43.18 85.09 0)
@@
 			)
 		)
-		(property "Manufacturer Part Number" "C1206C104K5RACTU"
+		(property "Manufacturer Part Number" ""
 			(at 91.44 133.35 0)
 			(hide yes)
@@
 			)
 		)
-		(property "Vendor Part Number" "399-C1206C104K5RACTUCT-ND"
+		(property "Vendor Part Number" ""
 			(at 91.44 133.35 0)
 			(hide yes)
@@
 			)
 		)
-		(property "Manufacturer Part Number" "RMCF1206FT10K0"
+		(property "Manufacturer Part Number" ""
 			(at 293.37 87.63 0)
 			(hide yes)
@@
 			)
 		)
-		(property "Vendor Part Number" "RMCF1206FT10K0CT-ND"
+		(property "Vendor Part Number" ""
 			(at 293.37 87.63 0)
 			(hide yes)
@@
 			)
 		)
-		(property "Manufacturer Part Number" "RMCF1206FT10K0"
+		(property "Manufacturer Part Number" ""
 			(at 43.18 78.74 0)
 			(hide yes)
@@
 			)
 		)
-		(property "Vendor Part Number" "RMCF1206FT10K0CT-ND"
+		(property "Vendor Part Number" ""
 			(at 43.18 78.74 0)
 			(hide yes)
