File: pcb/shift_registers.kicad_sch (KiCad schematic)
At the start: 5 parts, among them U23 74AHC595, U24 74AHC595, U25 74AHC595, U26 74AHC595, U27 74AHC595

Commit message: fix
Parts:
- added U28: ISO7760DW, Package_SO:SOIC-16W_7.5x10.3mm_P1.27mm, symbol Isolator:ISO7760DW
Connections:
- net +3.3V: now also U28.1 (Vcc1)
- net GND: now also U28.8 (GND1)
- new net +5V ISO: U28.16 (Vcc2)
- new net NGND: U28.9 (GND2)
- new net PWM_1: U28.15 (OUTA)
- new net PWM_2: U28.14 (OUTB)
- new net PWM_3: U28.13 (OUTC)
- new net PWM_4: U28.12 (OUTD)
- new net PWM_5: U28.11 (OUTE)
- new net PWM_6: U28.10 (OUTF)
- new net PWM_IN_1: U28.2 (INA)
- new net PWM_IN_2: U28.3 (INB)
- new net PWM_IN_3: U28.4 (INC)
- new net PWM_IN_4: U28.5 (IND)
- new net PWM_IN_5: U28.6 (INE)
- new net PWM_IN_6: U28.7 (INF)
Other:
- sheet Digit Tube & Driver 1 ports: added PWM; removed none
- sheet Digit Tube & Driver 2 ports: added PWM; removed none
- sheet Digit Tube & Driver 3 ports: added PWM; removed none
- sheet Digit Tube & Driver 4 ports: added PWM; removed none
- sheet Digit Tube & Driver 5 ports: added PWM; removed none
- sheet Digit Tube & Driver 6 ports: added PWM; removed none
- moved on the sheet: U26, U27

Commit message: w
Parts:
- U23, U24, U25, U26, U27: footprint (none) -> Package_SO:SOIC-16_3.9x9.9mm_P1.27mm
Changed lines of the file:
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@@
 			)
 		)
-		(property "Footprint" ""
+		(property "Footprint" "Package_SO:SOIC-16_3.9x9.9mm_P1.27mm"
 			(at 270.51 128.27 0)
 			(hide yes)
@@
 			)
 		)
-		(property "Footprint" ""
+		(property "Footprint" "Package_SO:SOIC-16_3.9x9.9mm_P1.27mm"
 			(at 269.24 59.69 0)
 			(hide yes)
@@
 			)
 		)
-		(property "Footprint" ""
+		(property "Footprint" "Package_SO:SOIC-16_3.9x9.9mm_P1.27mm"
 			(at 142.24 59.69 0)
 			(hide yes)
@@
 			)
 		)
-		(property "Footprint" ""
+		(property "Footprint" "Package_SO:SOIC-16_3.9x9.9mm_P1.27mm"
 			(at 140.97 196.85 0)
 			(hide yes)
@@
 			)
 		)
-		(property "Footprint" ""
+		(property "Footprint" "Package_SO:SOIC-16_3.9x9.9mm_P1.27mm"
 			(at 140.97 128.27 0)
 			(hide yes)
